File: kicad/zynq_card.kicad_sch (KiCad schematic)
At the start: 0 parts

Commit message: Phase 2: sheets 12-13 (ADC, connectors) + pin-plan netlist check
- Sheet 12: Ti135 ADC chain (SN74LV4051A checked against SCLS428K, OPA365,
  ADS7056 with AVDD on 3V3_analog and DVDD on 3V3), selects/SPI straight to bank 33.
- Sheet 13: J3 (baseboard J11 numbering, pin-plan notes asserted) with 32 x 10 k
  pull-downs, J5 LCD/touch, J2 console via SN74AVC4T774 (per-bit direction),
  I2C0 4.7 k pull-ups to 1V8 (no EEPROM for now).
- tools/check_pinplan_netlist.py: every PL and MIO signal on its ball: 0 failures.
- ERC: 4 expected pin_to_pin ties; block check 0 failures.

Co-Authored-By: Claude Opus 5.5 <noreply@anthropic.com>
Other:
- sheet 12 adc ports: added adbsel0, adbsel1, adbsel2, adc_cs_n, adc_sclk, adc_sdo, isoada1, isoada2, isoada3; removed none
- sheet 13 connectors ports: added adasel0_iso, adasel1_iso, adasel2_iso, adclk_dab, adclk_iso, clk1_iso, cs1_iso, dab_pwm_hi_sec, dab_pwm_lo_sec, dab_pwm_pri_hi_iso, dab_pwm_pri_lo_iso, gpio_bypass_rly_iso, gpio_bypass_rly_isolated, i2c_scl, i2c_sda, inu_adclk, isoada1, isoada2, isoada3, lcd_cs_n, lcd_dc, lcd_led, lcd_miso, lcd_mosi, lcd_reset_n, lcd_sck, mdata_dab, mdata_inu, mdata_iso, pwm_g1_iso, pwm_g2_iso, pwm_g3_iso, pwm_g4_iso, pwm_q5, pwm_q6, pwm_q7, pwm_q8, pwm_trans1_iso, pwm_trans2_iso, pwm_trans3_iso, pwm_trans4, pwm_trans5, pwm_trans6, sdata1_iso, t_clk, t_cs_n, t_din, t_do, t_irq, uart_rx, uart_tx; removed none
