File: kicad/zynq_card.kicad_pcb (KiCad board)
At the start: 8 copper layers, 76 x 65.1 mm, 309 parts, among them J1 JTAG 3V3, J2 UART 3V3, J3 2x19 1.27mm socket (bottom), J5 LCD 1x14 2.54mm, J6 2x3 1.27mm (bottom), J9 HR911130A, U1001 THGAMVG7T13BAIL, U1201 SN74LV4051APWR, U1202 OPA365AIDBVR, U1203 ADS7056IRUGR, U1301 SN74AVC4T774RSVR, U15 MT41K256M16TW-107:P, U16 MT41K256M16TW-107:P, U20 XC7Z020-1CLG484I, U301 TLV62585PDRLR, U311 TLV62585PDRLR, U321 TLV62585PDRLR, U331 TLV62585PDRLR, U341 NCP163ASN330T1G, U401 TPS3808G01DBVR, U601 SN74AVC4T774RSVR, U8 TPS51200DRCR, U801 IS25WP128-RHLE, U901 RTL8211FDI-CG, U902 74LVC1G07GW, Y701 33.333MHz, Y901 25MHz

Commit message: Phase 3 step 2: block copper import
tools/import_block.py copies juliancoy's SoC + DDR3 copper at pose A,
nets by pad, and makes the copper side of REUSE_LOG E3 and E5-E9.
Board-wide rail pours are clipped to the block; GND planes use the
source's fill settings. tools/check_block_copper.py: all 82 block
signal nets identical to the source except E3. ddr3_review.py on
both DRAMs: same lengths and vias, all PASS derated.

Co-Authored-By: Claude Opus 5.5 <noreply@anthropic.com>
Parts:
- added H1: MountingHole_3.2mm_M3, MountingHole:MountingHole_3.2mm_M3, F.Cu at (178.9, 101.9)
- added H2: MountingHole_3.2mm_M3, MountingHole:MountingHole_3.2mm_M3, F.Cu at (149.1, 72.1)
- C100, C101, C102, C103, C104, C105, C106, C11, C114, C116, C117, C118, C119, C121, C122, C125, C126, C127, C128, C129, C130, C131, C14, C15, C17, C18, C19, C20, C23, C24, C26, C28, C29, C30, C31, C33, C34, C4, C46, C47, C5, C50, C55, C57, C59, C61, C65, C67, C8, C9, C93, C98, D7, FB1, R10, R101, R102, R25, R49, R50, R51, R52, R53, R54, R55, R56, R57, R58, R59, R60, R61, R62, R63, R64, R65, R66, R67, R68, R69, R70, R71, R72, R74, R75, R9, U8: moved to B.Cu
- moved R62 214.8 mm to (157.4, 56.5)
- moved R61 212.0 mm to (156.9, 60.0), turned to -90 degrees
- moved R59 206.9 mm to (154.9, 54.6), turned to 90 degrees
- moved R60 205.9 mm to (159.4, 55.9), turned to 180 degrees
- moved R57 200.7 mm to (154.4, 56.6), turned to 180 degrees
- moved R58 197.2 mm to (161.3, 55.9)
- moved R55 194.4 mm to (154.0, 58.2), turned to 180 degrees
- moved R56 188.9 mm to (162.8, 56.9)
- moved R53 182.1 mm to (159.4, 56.8), turned to 180 degrees
- moved R54 182.1 mm to (162.9, 57.8)
- moved R52 181.8 mm to (156.3, 57.5), turned to 180 degrees
- moved R51 176.2 mm to (158.7, 58.3), turned to 180 degrees
- moved R50 175.7 mm to (156.0, 61.1), turned to 90 degrees
- moved R25 169.0 mm to (145.5, 59.0)
- moved R102 168.0 mm to (142.9, 57.6), turned to 90 degrees
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Routing:
- net GND: track 0.00 -> 80.4 mm, vias 0 -> 157
- net /01 ddr3/VREF: track 0.00 -> 69.4 mm, vias 0 -> 8
- net DDR3_A3: track 0.00 -> 53.7 mm, vias 0 -> 3
- net DDR3_DRST#: track 0.00 -> 53.6 mm, vias 0 -> 3
- net DDR3_A5: track 0.00 -> 52.8 mm, vias 0 -> 3
- net DDR3_BA2: track 0.00 -> 52.4 mm, vias 0 -> 3
- net DDR3_A1: track 0.00 -> 52.3 mm, vias 0 -> 3
- net DDR3_CAS#: track 0.00 -> 52.1 mm, vias 0 -> 3
- net DDR3_A10: track 0.00 -> 52.0 mm, vias 0 -> 3
- net DDR3_A0: track 0.00 -> 51.9 mm, vias 0 -> 3
- net DDR3_A7: track 0.00 -> 51.5 mm, vias 0 -> 3
- net DDR3_A2: track 0.00 -> 51.5 mm, vias 0 -> 3
- net DDR3_BA0: track 0.00 -> 51.5 mm, vias 0 -> 3
- net DDR3_A6: track 0.00 -> 50.8 mm, vias 0 -> 3
- net DDR3_A4: track 0.00 -> 50.7 mm, vias 0 -> 3
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- added copper zone on In4.Cu, net /05 soc_power/VCCAUX
- added copper zone on In6.Cu, net /05 soc_power/VCCAUX
- added copper zone on In6.Cu, net 1V0
- added copper zone on B.Cu, net 1V35
- added copper zone on F.Cu, net 1V35
- added copper zone on B.Cu, net 1V8
- added copper zone on In2.Cu, net 1V8
- added copper zone on In4.Cu, net 1V8
- added copper zone on In6.Cu, net 3V3
- added copper zone on B.Cu, net DDR3_VTT
- added copper zone on F.Cu, net GND
- added copper zone on In1.Cu, net GND
- added copper zone on In3.Cu, net GND
- added copper zone on In5.Cu, net GND

Commit message: Phase 3 steps 3-4: pose trials, rough placement at pose A0
- placement/: the KiCadRoutingTools inputs ported from the Ti135 card (groups,
  B.Cu TLV62585 templates, flip_bottom, fix_intent with the block and heatsink
  keep-outs, prep.sh), plus pose_trial.sh / pose_chain.txt for the pose trials.
- Pose trials: A0 29 open nets, Aw 32, Ae 28, B0 36, B1 36 (A beats B). The
  router was allowed to rip block copper in these runs; pose_trial.sh now sets
  KICAD_RIP_PREEXISTING=0 and the clean rerun is still to do.
- Rough placement on the board: A0's best seed, then the SoC decaps in a second
  run. DRC parity 0, no courtyard/clearance errors; block copper check 0.
- QSPI (MIO1-6) cannot route at any pose without juliancoy's F.Cu escapes:
  logged as a new block item.
- tools/apply_placement.py (ported; never moves a locked part).
- import_block/board_setup take P2K_PCB; import copies the trial project after
  the save and refuses a block off the board; check_block_copper picks block
  parts as the import does; build_pcb.sh --rebuild keeps the placement.

Co-Authored-By: Claude Opus 5.5 <noreply@anthropic.com>
Parts:
- C201, C202, C203, C301, C302, C303, C304, C311, C312, C313, C321, C322, C323, C331, C332, C333, C501, C502, C503, C504, C505, C506, C507, C508, C509, C510, C511, C512, C513, C514, C515, C516, C517, C518, C519, C520, C521, C522, C523, C524, C525, C526, C527, C528, C529, FB501, L301, L311, L321, L331, R301, R302, R311, R312, R321, R322, R331, R332, U301, U311, U321, U331: moved to B.Cu
- moved R932 232.1 mm to (135.5, 95.8), turned to 90 degrees
- moved R933 231.9 mm to (138.2, 99.3), turned to 90 degrees
- moved R930 226.3 mm to (136.8, 88.3), turned to 90 degrees
- moved R928 223.1 mm to (139.4, 71.1), turned to 90 degrees
- moved R925 217.3 mm to (137.2, 67.2), turned to 180 degrees
- moved R924 209.9 mm to (138.5, 75.0)
- moved RN1308 197.2 mm to (137.8, 63.5), turned to 90 degrees
- moved R920 196.9 mm to (141.0, 70.6)
- moved R931 195.8 mm to (188.3, 54.5), turned to 90 degrees
- moved R912 192.2 mm to (141.0, 74.3), turned to 90 degrees
- moved R909 189.4 mm to (136.5, 68.9), turned to 90 degrees
- moved R910 187.2 mm to (138.5, 77.0), turned to -90 degrees
- moved R950 184.7 mm to (199.1, 77.3)
- moved R927 181.9 mm to (185.9, 62.8), turned to -90 degrees
- moved RN1304 181.1 mm to (137.8, 72.4), turned to 180 degrees
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