File: kicad/zynq_card.kicad_pcb (KiCad board)
At the start: 8 copper layers, 76 x 65.1 mm, 311 parts, among them J1 JTAG 3V3, J2 UART 3V3, J3 2x19 1.27mm socket (bottom), J5 LCD 1x14 2.54mm, J6 2x3 1.27mm (bottom), J9 HR911130A, U1001 THGAMVG7T13BAIL, U1201 SN74LV4051APWR, U1202 OPA365AIDBVR, U1203 ADS7056IRUGR, U1301 SN74AVC4T774RSVR, U15 MT41K256M16TW-107:P, U16 MT41K256M16TW-107:P, U20 XC7Z020-1CLG484I, U301 TLV62585PDRLR, U311 TLV62585PDRLR, U321 TLV62585PDRLR, U331 TLV62585PDRLR, U341 NCP163ASN330T1G, U401 TPS3808G01DBVR, U601 SN74AVC4T774RSVR, U8 TPS51200DRCR, U801 IS25WP128-RHLE, U901 RTL8211FDI-CG, U902 74LVC1G07GW, Y701 33.333MHz, Y901 25MHz

Commit message: Phase 3 step 4: analog copied from the Ti135 card, KRT re-place with claims; QSPI escapes (E10)
- tools/place_analog.py (ported from the Ti135 card): the ADC chain and the
  3V3_analog LDO take the Ti135 card's final positions from J3 (its copy of
  the Agilex 5 card, same outline and circuit); the four parts that would sit
  in our block area go to the nearest free spot. The J3 pull-down arrays go
  to B.Cu in a column beside J3. All locked.
- placement/touchup.py: lock all but a set of parts and give each a proximity
  claim to the chip it serves. KRT re-placed the other 143 parts with claims
  (claim weight 20): median distance to their pins 11.1 -> 4.0 mm, Ethernet
  spread 65 -> 23 mm. DRC parity 0, no courtyard/clearance errors; block
  copper check 0 failures.
- REUSE_LOG E10: import_block copies juliancoy's F.Cu escapes of the six QSPI
  balls (walled in by byte-0 DDR copper) to their vias.
- Pose trials rerun with the block copper protected: Ae 26, Aw 32, A0 35,
  B0 37, B1 43 open nets; A beats B. pose_trial.sh sets KICAD_PYTHON too.
- prep.sh copies its intent back only for the real board.
- LAYOUT_PLAN/STATUS: results, the KRT survey, the hand-fix list.

Co-Authored-By: Claude Opus 5.5 <noreply@anthropic.com>
Parts:
- RN1301, RN1302, RN1303, RN1304, RN1305, RN1306, RN1307, RN1308: moved to B.Cu
- moved RN1307 78.5 mm to (137.9, 56.6), turned to -90 degrees
- moved RN1306 70.2 mm to (137.9, 59.3), turned to -90 degrees
- moved C922 69.1 mm to (205.0, 74.6), turned to 0 degrees
- moved R909 68.6 mm to (202.9, 86.2)
- moved R930 67.8 mm to (204.5, 83.8), turned to 180 degrees
- moved C932 67.4 mm to (204.0, 82.1)
- moved C940 67.4 mm to (206.0, 80.6), turned to 0 degrees
- moved C930 67.0 mm to (202.1, 81.5), turned to 0 degrees
- moved FB901 66.7 mm to (203.6, 76.8), turned to 90 degrees
- moved C921 66.2 mm to (202.2, 73.7), turned to 90 degrees
- moved C935 65.1 mm to (202.4, 82.6), turned to 0 degrees
- moved R933 65.0 mm to (197.3, 72.2)
- moved U902 64.7 mm to (195.3, 73.5), turned to 0 degrees
- moved R925 64.5 mm to (200.1, 81.5)
- moved C941 63.2 mm to (203.0, 84.1), turned to -90 degrees
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Routing:
- net /qspi_cs_n: track 0.00 -> 2.91 mm, vias 0 -> 1
- net /qspi_sclk: track 0.00 -> 1.27 mm, vias 0 -> 1
- net /qspi_io2: track 0.00 -> 0.57 mm, vias 0 -> 1
- net /qspi_io3: track 0.00 -> 0.57 mm, vias 0 -> 1
- net /qspi_io1: track 0.00 -> 0.57 mm, vias 0 -> 1
- net /qspi_io0: track 0.00 -> 0.57 mm, vias 0 -> 1
