File: kicad/zynq_card.kicad_pcb (KiCad board)
At the start: 8 copper layers, 76 x 65.1 mm, 311 parts, among them J1 JTAG 3V3, J2 UART 3V3, J3 2x19 1.27mm socket (bottom), J5 LCD 1x14 2.54mm, J6 2x3 1.27mm (bottom), J9 HR911130A, U1001 THGAMVG7T13BAIL, U1201 SN74LV4051APWR, U1202 OPA365AIDBVR, U1203 ADS7056IRUGR, U1301 SN74AVC4T774RSVR, U15 MT41K256M16TW-107:P, U16 MT41K256M16TW-107:P, U20 XC7Z020-2CLG484I, U301 TLV62585PDRLR, U311 TLV62585PDRLR, U321 TLV62585PDRLR, U331 TLV62585PDRLR, U341 NCP163ASN330T1G, U401 TPS3808G01DBVR, U601 SN74AVC4T774RSVR, U8 TPS51200DRCR, U801 IS25WP128-RHLE, U901 RTL8211FDI-CG, U902 74LVC1G07GW, Y701 33.333MHz, Y901 25MHz

Commit message: E13: C99 out from under the heatsink base; phase 3 layer renders done
C99 (1V35 bulk, 100 uF 1210, 2.7 mm) sat 1.2-1.4 mm inside the heatsink
base, where nothing may be taller than the package. tools/block_e13.py
(run by build_pcb.sh --rebuild after block_e1.py) moves it 2.2 mm north;
its GND via stays (DDR3 copper on every inner layer under the moved pad)
and a 0.3 mm F.Cu track joins pad 2 to it. DRC unchanged, block copper
check 0 failures, a --rebuild reproduces the board.

Co-Authored-By: Claude Opus 5.5 <noreply@anthropic.com>
Parts:
- moved C99 2.20 mm to (156.9, 72.6)
Routing:
- net GND: track 81.1 -> 83.3 mm
