File: kicad/01_ddr3.kicad_sch (KiCad schematic)
At the start: 62 parts, among them U15 MT41K256M16TW-107:P, U16 MT41K256M16TW-107:P, U20 xc7z020clg484, U8 TPS51200DRCR

Commit message: LCSC numbers for every BOM part (tools/set_lcsc.py); FB1 as 0 R; U20 = XC7Z020-2CLG484I
tools/set_lcsc.py (run by build_schematic.sh) writes the LCSC field by BOM line: JLC basic parts where there is one,
juliancoy's Murata/Yageo passives bought as basic equivalents (REUSE_LOG E11). FB1, the E5 0 R jumper, gets
0603WAF0000T5E / C21189 (its MPN still named the bead). U20: -2 or -3 speed, any temperature grade (user):
XC7Z020-2CLG484I, C157624. Connectors J1/J2/J3/J5/J6/J9 hand-soldered (no LCSC, skipped in the JLC files).
ERC unchanged (4 intended pin_to_pin), block netlist 0 failures, board rebuilt: parity 0, block copper 0 failures.

Co-Authored-By: Claude Opus 5.5 <noreply@anthropic.com>
Parts:
- C100, C127: LCSC (none) -> C23733; MFR Murata -> (none); MPN GRM155R60G475ME47D -> CL05A475MP5NRNC; SPN 490-11980-1-ND -> (none); SPR Digikey -> (none)
- C101, C102, C103, C104: LCSC (none) -> C47339; MFR Yageo -> (none); MPN CC0402KRX5R5BB474 -> CL05A474KP5NNNC; SPN 311-1684-1-ND -> (none); SPR Digikey -> (none)
- C105, C106, C109, C110, C93, C98: LCSC (none) -> C15195; MFR Murata -> (none); MPN GRM155R71H103KA88J -> CL05B103KB5NNNC; SPN 490-6351-1-ND -> (none); SPR Digikey -> (none); SPURL - -> (none)
- C125, C126, C128, C129, C130: LCSC (none) -> C19702; MFR Murata -> (none); MPN GRM188R61A106KE69J -> CL10A106KP8NNNC; SPN 490-14372-1-ND -> (none); SPR Digikey -> (none)
- C131, C94, C95, C96, C97: LCSC (none) -> C1525; MFR Yageo -> (none); MPN CC0402KRX7R6BB104 -> CL05B104KO5NNNC; SPN 311-1345-1-ND -> (none); SPR Digikey -> (none)
- C99: LCSC (none) -> C49066; MFR TAIYO YUDEN -> (none); MPN JMK325ABJ107MM-P -> CL32A107MQVNNNE; SPN 587-4313-1-ND -> (none); SPR Digikey -> (none)
- D7: LCSC (none) -> C435849
- R101: LCSC (none) -> C25741; MFR Yageo -> (none); MPN RC0402FR-07100KL -> 0402WGF1003TCE; SPN 311-100KLRTR-ND -> (none); SPR Digikey -> (none)
- R102: LCSC (none) -> C140202; MFR Yageo -> (none); MPN RC0402FR-07150RL -> RC-02K1500FT; SPN 311-150LRTR-ND -> (none); SPR Digikey -> (none)
- R25: LCSC (none) -> C705630
- R46, R49: LCSC (none) -> C114755
- R47, R48: LCSC (none) -> C25744; MFR Yageo -> (none); MPN RC0402FR-0710KL -> 0402WGF1002TCE; SPN 311-10.0KLRCT-ND -> (none); SPR Digikey -> (none); SPURL - -> (none)
- R50, R75, R76: LCSC (none) -> C185392
- R51, R52, R53, R54, R55, R56, R57, R58, R59, R60, R61, R62, R63, R64, R65, R66, R67, R68, R69, R70, R71, R72, R73: LCSC (none) -> C274892
- R74: LCSC (none) -> C25900; MFR Yageo -> (none); MPN RC0402JR-074K7L -> 0402WGF4701TCE; SPN 311-4.7KJRCT-ND -> (none); SPR Digikey -> (none); SPURL - -> (none)
- U20: value xc7z020clg484 -> XC7Z020-2CLG484I; LCSC (none) -> C157624; MPN XC7Z020-1CLG484C -> XC7Z020-2CLG484I
- U8: LCSC (none) -> C34771
