File: kicad/02_pwr_input.kicad_sch (KiCad schematic)
At the start: 0 parts

Commit message: Phase 2: sheets 2-4 (power input, rails, sequencing + PS_POR_B supervisor)
Sheet 2: J6 (baseboard J12) to 5V0/GND with PWR_FLAGs and the Ti135 input bulk.
Sheet 3: 4 x TLV62585 (1V0, 1V8, 3V3, 1V35) from the Ti135 cell (_power.py) and
the NCP163 3V3_analog LDO.
Sheet 4: enable chain 1V0 -> 1V8 -> 3V3 + 1V35 -> DDR3_VTT_EN (wired PG AND)
and a TPS3808G01 onto ps_por_n: SENSE on 1V0 (0.895 V), CT = VDD (300 ms),
which keeps PS_POR_B release outside every DS187 Table 23 lockdown window.
Closes the lockdown-window [verify] item. ERC: rails driven; block check 0 failures.

Co-Authored-By: Claude Opus 5.5 <noreply@anthropic.com>
Parts:
- added C201: 47u, Capacitor_SMD:C_1206_3216Metric, symbol zynq_card:C
- added C202: 22u, Capacitor_SMD:C_0805_2012Metric, symbol zynq_card:C
- added C203: 100n, Capacitor_SMD:C_0402_1005Metric, symbol zynq_card:C
- added J6: 2x3 1.27mm (bottom), Connector_PinSocket_1.27mm:PinSocket_2x03_P1.27mm_Vertical, symbol zynq_card:Conn_02x03_Odd_Even
Connections:
- new net 5V0: C201.1, C202.1, C203.1, J6.2 (Pin_2), J6.4 (Pin_4), J6.6 (Pin_6)
- new net GND: C201.2, C202.2, C203.2, J6.1 (Pin_1), J6.3 (Pin_3), J6.5 (Pin_5)
Other:
- note added: "GND: the card's only ground (baseboard ISOGND)"
- note added: "Input bulk at J6 (the regulators have their own 10u)."
- note added: "J6 = baseboard J12 (2x3 1.27 mm socket on B.Cu, MECHANICAL.md): 5V0 = baseboard 5V_ISOL, GND = ISOGND. Supply budget: POWER_BUDGET.md (0.89 A typ / 1.44 A high; needs the baseboard U8 upgrade to 1.5-2 A)."

Commit message: LCSC numbers for every BOM part (tools/set_lcsc.py); FB1 as 0 R; U20 = XC7Z020-2CLG484I
tools/set_lcsc.py (run by build_schematic.sh) writes the LCSC field by BOM line: JLC basic parts where there is one,
juliancoy's Murata/Yageo passives bought as basic equivalents (REUSE_LOG E11). FB1, the E5 0 R jumper, gets
0603WAF0000T5E / C21189 (its MPN still named the bead). U20: -2 or -3 speed, any temperature grade (user):
XC7Z020-2CLG484I, C157624. Connectors J1/J2/J3/J5/J6/J9 hand-soldered (no LCSC, skipped in the JLC files).
ERC unchanged (4 intended pin_to_pin), block netlist 0 failures, board rebuilt: parity 0, block copper 0 failures.

Co-Authored-By: Claude Opus 5.5 <noreply@anthropic.com>
Parts:
- C201: LCSC (none) -> C96123
- C202: LCSC (none) -> C45783
- C203: LCSC (none) -> C1525
Changed lines of the file:
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@@
+			)
+		)
+		(property "LCSC" "C96123"
+			(at 88.9 66.04 0)
+			(effects
+				(font
+					(size 1.27 1.27)
+				)
+				(hide yes)
 			)
 		)
@@
 			)
 		)
+		(property "LCSC" "C45783"
+			(at 99.06 66.04 0)
+			(effects
+				(font
+					(size 1.27 1.27)
+				)
+				(hide yes)
+			)
+		)
 		(property "Description" "Unpolarized capacitor"
 			(at 99.06 66.04 0)
@@
 			(at 109.22 66.04 0)
 			(effects
+				(font
+					(size 1.27 1.27)
+				)
+				(hide yes)
+			)
+		)
+		(property "LCSC" "C1525"
+			(at 109.22 66.04 0)
+			(effects
