File: kicad/03_pwr_rails.kicad_sch (KiCad schematic)
At the start: 0 parts

Commit message: Phase 2: sheets 2-4 (power input, rails, sequencing + PS_POR_B supervisor)
Sheet 2: J6 (baseboard J12) to 5V0/GND with PWR_FLAGs and the Ti135 input bulk.
Sheet 3: 4 x TLV62585 (1V0, 1V8, 3V3, 1V35) from the Ti135 cell (_power.py) and
the NCP163 3V3_analog LDO.
Sheet 4: enable chain 1V0 -> 1V8 -> 3V3 + 1V35 -> DDR3_VTT_EN (wired PG AND)
and a TPS3808G01 onto ps_por_n: SENSE on 1V0 (0.895 V), CT = VDD (300 ms),
which keeps PS_POR_B release outside every DS187 Table 23 lockdown window.
Closes the lockdown-window [verify] item. ERC: rails driven; block check 0 failures.

Co-Authored-By: Claude Opus 5.5 <noreply@anthropic.com>
Parts:
- added C301, C311, C321, C331: 10u, Capacitor_SMD:C_0805_2012Metric, symbol zynq_card:C
- added C302, C303, C312, C322, C332: 22u, Capacitor_SMD:C_0805_2012Metric, symbol zynq_card:C
- added C304, C313, C323, C333: 22p, Capacitor_SMD:C_0402_1005Metric, symbol zynq_card:C
- added C341, C342: 1u, Capacitor_SMD:C_0402_1005Metric, symbol zynq_card:C
- added L301, L311, L321, L331: 1u, Inductor_SMD:L_Coilcraft_XxL4020, symbol zynq_card:L_Power
- added R301: 66.5k, Resistor_SMD:R_0402_1005Metric, symbol zynq_card:R
- added R302, R312, R322, R332: 100k, Resistor_SMD:R_0402_1005Metric, symbol zynq_card:R
- added R311: 200k, Resistor_SMD:R_0402_1005Metric, symbol zynq_card:R
- added R321: 453k, Resistor_SMD:R_0402_1005Metric, symbol zynq_card:R
- added R331: 124k, Resistor_SMD:R_0402_1005Metric, symbol zynq_card:R
- added U301, U311, U321, U331: TLV62585PDRLR, Package_TO_SOT_SMD:SOT-563, symbol zynq_card:TLV62585PDRL
- added U341: NCP163ASN330T1G, Package_TO_SOT_SMD:SOT-23-5, symbol zynq_card:NCP163ASN330T1G
Connections:
- new net: L301.1, U301.2 (SW)
- new net: C304.2, R301.2, R302.1, U301.5 (FB)
- new net: C313.2, R311.2, R312.1, U311.5 (FB)
- new net: C333.2, R331.2, R332.1, U331.5 (FB)
- new net: L331.1, U331.2 (SW)
- new net: L321.1, U321.2 (SW)
- new net: C323.2, R321.2, R322.1, U321.5 (FB)
- new net: L311.1, U311.2 (SW)
- new net 1V0: C302.1, C303.1, C304.1, L301.2, R301.1
- new net 1V35: C332.1, C333.1, L331.2, R331.1
- new net 1V8: C312.1, C313.1, L311.2, R311.1
- new net 3V3: C322.1, C323.1, L321.2, R321.1
- new net 3V3_analog: C342.1, U341.5 (VOUT)
- new net 5V0: C301.1, C311.1, C321.1, C331.1, C341.1, U301.3 (VIN), U301.4 (EN), U311.3 (VIN), U321.3 (VIN), U331.3 (VIN), U341.1 (VIN), U341.3 (EN)
- new net DDR3_VTT_EN: U321.6 (PG), U331.6 (PG)
- new net GND: C301.2, C302.2, C303.2, C311.2, C312.2, C321.2, C322.2, C331.2, C332.2, C341.2, C342.2, R302.2, R312.2, R322.2, R332.2, U301.1 (GND), U311.1 (GND), U321.1 (GND), U331.1 (GND), U341.2 (GND)
- new net pg_1v0: U301.6 (PG), U311.4 (EN)
- new net pg_1v8: U311.6 (PG), U321.4 (EN), U331.4 (EN)
- no-connect marks 0 -> 1
Other:
- note added: "1V0: VCCPINT, VCCINT, VCCBRAM (2.40 A high)"
- note added: "1V35: VCCO_DDR, DDR3L, TPS51200 VLDOIN (0.97 A)"
- note added: "1V8: VCCPAUX, VCCPLL, VCCAUX, VCCO_MIO, bank 0 (0.40 A)"
- note added: "3V3: HR banks 13/33/34/35, PHY, eMMC, LCD (0.49 A)"
- note added: "3V3_analog: LDO from 5V0 for the ADC block (sheet 12), always on (not in the SoC sequence)."
- note added: "Order (sheet 4): 1V0 -> 1V8 (VCCPAUX, VCCPLL, VCCAUX, VCCO_MIO, bank 0) -> 3V3 (HR banks) and 1V35 (VCCO_DDR, DDR3L) -> DDR3_VTT_EN (TPS51200, sheet 1) -> U401 (300 ms) -> PS_POR_B. 1V8 is up before 3V3 starts: VCCO - VCCAUX <= 2.625 V."

Commit message: LCSC numbers for every BOM part (tools/set_lcsc.py); FB1 as 0 R; U20 = XC7Z020-2CLG484I
tools/set_lcsc.py (run by build_schematic.sh) writes the LCSC field by BOM line: JLC basic parts where there is one,
juliancoy's Murata/Yageo passives bought as basic equivalents (REUSE_LOG E11). FB1, the E5 0 R jumper, gets
0603WAF0000T5E / C21189 (its MPN still named the bead). U20: -2 or -3 speed, any temperature grade (user):
XC7Z020-2CLG484I, C157624. Connectors J1/J2/J3/J5/J6/J9 hand-soldered (no LCSC, skipped in the JLC files).
ERC unchanged (4 intended pin_to_pin), block netlist 0 failures, board rebuilt: parity 0, block copper 0 failures.

Co-Authored-By: Claude Opus 5.5 <noreply@anthropic.com>
Parts:
- C301, C311, C321, C331: LCSC (none) -> C15850
- C302, C303, C312, C322, C332: LCSC (none) -> C45783
- C304, C313, C323, C333: LCSC (none) -> C1555
- C341, C342: LCSC (none) -> C52923
- R301: LCSC (none) -> C2998095
- R302, R312, R322, R332: LCSC (none) -> C25741
- R311: LCSC (none) -> C25764
- R321: LCSC (none) -> C27009
- R331: LCSC (none) -> C2933070
- U341: LCSC (none) -> C603656
Changed lines of the file:
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@@
 			)
 		)
+		(property "LCSC" "C15850"
+			(at 38.1 64.77 0)
+			(effects
+				(font
+					(size 1.27 1.27)
+				)
+				(hide yes)
+			)
+		)
 		(property "Description" "Unpolarized capacitor"
 			(at 38.1 64.77 0)
@@
 			)
 		)
+		(property "LCSC" "C2998095"
+			(at 104.14 64.77 0)
+			(effects
+				(font
+					(size 1.27 1.27)
+				)
+				(hide yes)
+			)
+		)
 		(property "Description" "Resistor"
 			(at 104.14 64.77 0)
@@
 			)
 		)
+		(property "LCSC" "C25741"
+			(at 104.14 74.93 0)
+			(effects
+				(font
+					(size 1.27 1.27)
+				)
+				(hide yes)
+			)
+		)
 		(property "Description" "Resistor"
 			(at 104.14 74.93 0)
@@
 			)
 		)
+		(property "LCSC" "C1555"
+			(at 118.11 64.77 0)
+			(effects
+				(font
+					(size 1.27 1.27)
+				)
+				(hide yes)
+			)
+		)
 		(property "Description" "Unpolarized capacitor"
 			(at 118.11 64.77 0)
@@
 			)
 		)
+		(property "LCSC" "C45783"
+			(at 129.54 64.77 0)
+			(effects
+				(font
+					(size 1.27 1.27)
+				)
+				(hide yes)
+			)
+		)
 		(property "Description" "Unpolarized capacitor"
 			(at 129.54 64.77 0)
@@
 			)
 		)
+		(property "LCSC" "C45783"
+			(at 139.7 64.77 0)
+			(effects
+				(font
+					(size 1.27 1.27)
+				)
+				(hide yes)
+			)
+		)
 		(property "Description" "Unpolarized capacitor"
 			(at 139.7 64.77 0)
@@
 			)
 		)
+		(property "LCSC" "C15850"
+			(at 177.8 64.77 0)
+			(effects
+				(font
+					(size 1.27 1.27)
+				)
+				(hide yes)
+			)
+		)
 		(property "Description" "Unpolarized capacitor"
 			(at 177.8 64.77 0)
@@
 			)
 		)
+		(property "LCSC" "C25764"
+			(at 243.84 64.77 0)
+			(effects
+				(font
+					(size 1.27 1.27)
+				)
+				(hide yes)
+			)
+		)
 		(property "Description" "Resistor"
 			(at 243.84 64.77 0)
@@
 			)
 		)
+		(property "LCSC" "C25741"
+			(at 243.84 74.93 0)
+			(effects
+				(font
+					(size 1.27 1.27)
+				)
+				(hide yes)
+			)
+		)
 		(property "Description" "Resistor"
 			(at 243.84 74.93 0)
@@
 			)
 		)
+		(property "LCSC" "C1555"
+			(at 257.81 64.77 0)
+			(effects
+				(font
+					(size 1.27 1.27)
+				)
+				(hide yes)
+			)
+		)
 		(property "Description" "Unpolarized capacitor"
 			(at 257.81 64.77 0)
@@
 			)
 		)
+		(property "LCSC" "C45783"
+			(at 269.24 64.77 0)
+			(effects
+				(font
+					(size 1.27 1.27)
+				)
+				(hide yes)
+			)
+		)
 		(property "Description" "Unpolarized capacitor"
 			(at 269.24 64.77 0)
@@
 			)
 		)
+		(property "LCSC" "C15850"
+			(at 38.1 143.51 0)
+			(effects
+				(font
+					(size 1.27 1.27)
+				)
+				(hide yes)
+			)
+		)
 		(property "Description" "Unpolarized capacitor"
 			(at 38.1 143.51 0)
@@
 			)
 		)
+		(property "LCSC" "C27009"
+			(at 104.14 143.51 0)
+			(effects
+				(font
+					(size 1.27 1.27)
+				)
+				(hide yes)
+			)
+		)
 		(property "Description" "Resistor"
 			(at 104.14 143.51 0)
@@
 			)
 		)
+		(property "LCSC" "C25741"
+			(at 104.14 153.67 0)
+			(effects
+				(font
+					(size 1.27 1.27)
+				)
+				(hide yes)
+			)
+		)
 		(property "Description" "Resistor"
 			(at 104.14 153.67 0)
@@
 			)
 		)
+		(property "LCSC" "C1555"
+			(at 118.11 143.51 0)
+			(effects
+				(font
+					(size 1.27 1.27)
+				)
+				(hide yes)
+			)
+		)
 		(property "Description" "Unpolarized capacitor"
 			(at 118.11 143.51 0)
@@
 			)
 		)
+		(property "LCSC" "C45783"
+			(at 129.54 143.51 0)
+			(effects
+				(font
+					(size 1.27 1.27)
+				)
+				(hide yes)
+			)
+		)
 		(property "Description" "Unpolarized capacitor"
 			(at 129.54 143.51 0)
@@
 			)
 		)
+		(property "LCSC" "C15850"
+			(at 177.8 143.51 0)
+			(effects
+				(font
+					(size 1.27 1.27)
+				)
+				(hide yes)
+			)
+		)
 		(property "Description" "Unpolarized capacitor"
 			(at 177.8 143.51 0)
@@
 			)
 		)
+		(property "LCSC" "C2933070"
+			(at 243.84 143.51 0)
+			(effects
+				(font
+					(size 1.27 1.27)
+				)
+				(hide yes)
+			)
+		)
 		(property "Description" "Resistor"
 			(at 243.84 143.51 0)
@@
 			)
 		)
+		(property "LCSC" "C25741"
+			(at 243.84 153.67 0)
+			(effects
+				(font
+					(size 1.27 1.27)
+				)
+				(hide yes)
+			)
+		)
 		(property "Description" "Resistor"
 			(at 243.84 153.67 0)
@@
 			)
 		)
+		(property "LCSC" "C1555"
+			(at 257.81 143.51 0)
+			(effects
+				(font
+					(size 1.27 1.27)
+				)
+				(hide yes)
+			)
+		)
 		(property "Description" "Unpolarized capacitor"
 			(at 257.81 143.51 0)
@@
 			)
 		)
+		(property "LCSC" "C45783"
+			(at 269.24 143.51 0)
+			(effects
+				(font
+					(size 1.27 1.27)
+				)
+				(hide yes)
+			)
+		)
 		(property "Description" "Unpolarized capacitor"
 			(at 269.24 143.51 0)
@@
 			)
 		)
+		(property "LCSC" "C603656"
+			(at 342.9 66.04 0)
+			(effects
+				(font
+					(size 1.27 1.27)
+				)
+				(hide yes)
+			)
+		)
 		(property "Description" "250mA low-noise LDO, 2.2V-5.5V input, 3.3V output, SOT-23-5"
 			(at 342.9 66.04 0)
@@
 			)
 		)
+		(property "LCSC" "C52923"
+			(at 322.58 71.12 0)
+			(effects
+				(font
+					(size 1.27 1.27)
+				)
+				(hide yes)
+			)
+		)
 		(property "Description" "Unpolarized capacitor"
 			(at 322.58 71.12 0)
@@
 			(at 358.14 71.12 0)
 			(effects
+				(font
+					(size 1.27 1.27)
+				)
+				(hide yes)
+			)
+		)
+		(property "LCSC" "C52923"
+			(at 358.14 71.12 0)
+			(effects
