File: kicad/04_pwr_seq.kicad_sch (KiCad schematic)
At the start: 0 parts

Commit message: Phase 2: sheets 2-4 (power input, rails, sequencing + PS_POR_B supervisor)
Sheet 2: J6 (baseboard J12) to 5V0/GND with PWR_FLAGs and the Ti135 input bulk.
Sheet 3: 4 x TLV62585 (1V0, 1V8, 3V3, 1V35) from the Ti135 cell (_power.py) and
the NCP163 3V3_analog LDO.
Sheet 4: enable chain 1V0 -> 1V8 -> 3V3 + 1V35 -> DDR3_VTT_EN (wired PG AND)
and a TPS3808G01 onto ps_por_n: SENSE on 1V0 (0.895 V), CT = VDD (300 ms),
which keeps PS_POR_B release outside every DS187 Table 23 lockdown window.
Closes the lockdown-window [verify] item. ERC: rails driven; block check 0 failures.

Co-Authored-By: Claude Opus 5.5 <noreply@anthropic.com>
Parts:
- added C401: 100n, Capacitor_SMD:C_0402_1005Metric, symbol zynq_card:C
- added R401, R402, R404: 100k, Resistor_SMD:R_0402_1005Metric, symbol zynq_card:R
- added R403: 121k, Resistor_SMD:R_0402_1005Metric, symbol zynq_card:R
- added U401: TPS3808G01DBVR, Package_TO_SOT_SMD:SOT-23-6, symbol zynq_card:TPS3808DBV
Connections:
- new net 1V0: R403.1
- new net 1V8: C401.1, U401.4 (CT), U401.6 (VDD)
- new net 5V0: R401.1, R402.1
- new net DDR3_VTT_EN: U401.3 (~{MR})
- new net GND: C401.2, R404.2, U401.2 (GND)
- new net pg_1v0: R401.2
- new net pg_1v8: R402.2
- new net por_sense: R403.2, R404.1, U401.5 (SENSE)
- new net ps_por_n: U401.1 (~{RESET})
Other:
- note added: "CT = VDD (1V8): t_D = 300 ms"
- note added: "DDR3_VTT_EN = PG(3V3) & PG(1V35), wired AND, pull-up R25 20k to 3V3 (sheet 1) = TPS51200 EN"
- note added: "Power-up (ZYNQ_PCB_NOTES.md §3): 5V0 -> 1V0 -> pg_1v0 -> 1V8 -> pg_1v8 -> 3V3 + 1V35 -> DDR3_VTT_EN (TPS51200 VTT) -> U401 TPS3808G01 (CT = VDD: 300 ms) -> ps_por_n (PS_POR_B). Each TLV62585 ramps in 0.9 ms (DS187: 0.2-50 ms). 300 ms keeps PS_POR_B release outside the DS187 Table 23 secure lockdown window in every boot configuration."
- note added: "SENSE divider: 1V0 < 0.895 V -> reset (asserted before VCCPINT reaches 0.80 V)"
- note added: "open drain; 10k pull-up to 1V8 is R608 on sheet 6"
- note added: "pg_1v0 = PG(1V0) -> EN of 1V8"
- note added: "pg_1v8 = PG(1V8) -> EN of 3V3 and 1V35"

Commit message: LCSC numbers for every BOM part (tools/set_lcsc.py); FB1 as 0 R; U20 = XC7Z020-2CLG484I
tools/set_lcsc.py (run by build_schematic.sh) writes the LCSC field by BOM line: JLC basic parts where there is one,
juliancoy's Murata/Yageo passives bought as basic equivalents (REUSE_LOG E11). FB1, the E5 0 R jumper, gets
0603WAF0000T5E / C21189 (its MPN still named the bead). U20: -2 or -3 speed, any temperature grade (user):
XC7Z020-2CLG484I, C157624. Connectors J1/J2/J3/J5/J6/J9 hand-soldered (no LCSC, skipped in the JLC files).
ERC unchanged (4 intended pin_to_pin), block netlist 0 failures, board rebuilt: parity 0, block copper 0 failures.

Co-Authored-By: Claude Opus 5.5 <noreply@anthropic.com>
Parts:
- C401: LCSC (none) -> C1525
- R401, R402, R404: LCSC (none) -> C25741
- R403: LCSC (none) -> C11693
- U401: LCSC (none) -> C19653
Changed lines of the file:
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@@
+			)
+		)
+		(property "LCSC" "C25741"
+			(at 55.88 57.15 0)
+			(effects
+				(font
+					(size 1.27 1.27)
+				)
+				(hide yes)
 			)
 		)
@@
 			)
 		)
+		(property "LCSC" "C25741"
+			(at 55.88 95.25 0)
+			(effects
+				(font
+					(size 1.27 1.27)
+				)
+				(hide yes)
+			)
+		)
 		(property "Description" "Resistor"
 			(at 55.88 95.25 0)
@@
 		(property "Datasheet" ""
 			(at 162.56 83.82 0)
+			(effects
+				(font
+					(size 1.27 1.27)
+				)
+				(hide yes)
+			)
+		)
+		(property "LCSC" "C19653"
+			(at 165.1 83.82 0)
 			(effects
 				(font
@@
 			)
 		)
+		(property "LCSC" "C11693"
+			(at 106.68 110.49 0)
+			(effects
+				(font
+					(size 1.27 1.27)
+				)
+				(hide yes)
+			)
+		)
 		(property "Description" "Resistor"
 			(at 106.68 110.49 0)
@@
 		)
 		(property "Datasheet" ""
+			(at 106.68 123.19 0)
+			(effects
+				(font
+					(size 1.27 1.27)
+				)
+				(hide yes)
+			)
+		)
+		(property "LCSC" "C25741"
 			(at 106.68 123.19 0)
 			(effects
@@
 			(at 193.04 66.04 0)
 			(effects
+				(font
+					(size 1.27 1.27)
+				)
+				(hide yes)
+			)
+		)
+		(property "LCSC" "C1525"
+			(at 193.04 66.04 0)
+			(effects
