File: kicad/05_soc_power.kicad_sch (KiCad schematic)
At the start: 0 parts

Commit message: Phase 2: sheet 5 (SoC power): U20 unit 9 and decoupling
- tools/sheets/_legacy.py: the KiCad 5 converter, shared by the block
  sheets; keep= takes a subset of a source sheet and prunes what no longer
  reaches a kept pin, cut= drops source wires, mirrored symbols supported.
  01_ddr3.py uses it and regenerates byte-identical
- tools/sheets/05_soc_power.py: U20 unit 9 and the 21 power.sch decaps in
  the block copper (source refs/positions), the 16 3V3 block caps juliancoy
  drew on other sheets, and C501-C529 + FB501 to meet UG933 Tables 3-1/3-2
- E5: VCCPLL through its own 120R bead + 10u + 470n; FB1 (juliancoy's
  VCCAUX bead) becomes a 0 ohm jumper. E6: C59/C122 on 1V8 (MIO banks).
  E7 planned: VCCO_MIO / VCCO_34/35 ball fan-out at the copper import
- Bank 0 stays at 1.8 V as on juliancoy: CFGBVS GND, JTAG 1.8 V; Vivado
  pin plan re-run with CONFIG_VOLTAGE 1.8 (DRC 0)
- check_block_netlist.py covers sheets 1 and 5 (99 parts, 555 pads,
  0 failures); gen_symbols adds 1V0/1V8, FerriteBead_Small, C_Polarized
- STATUS.md, REUSE_LOG.md, ZYNQ_PCB_NOTES.md updated

Co-Authored-By: Claude Opus 5.5 <noreply@anthropic.com>
Parts:
- added C11, C26, C33: 10uF, Capacitor_SMD:C_0603_1608Metric, symbol zynq_card:C_Small
- added C114, C122, C57, C59: 4.7uF, Capacitor_SMD:C_0402_1005Metric, symbol zynq_card:C
- added C116, C117, C118, C119, C121, C46, C47, C50, C55, C65: .47uF, Capacitor_SMD:C_0402_1005Metric, symbol zynq_card:C
- added C14, C15, C17, C18, C23, C29, C30, C31, C34, C4, C8: .47uF, Capacitor_SMD:C_0402_1005Metric, symbol zynq_card:C_Small
- added C19, C20, C24, C5, C9: 4.7uF, Capacitor_SMD:C_0402_1005Metric, symbol zynq_card:C_Small
- added C28: 100uF, Capacitor_SMD:C_1210_3225Metric, symbol zynq_card:C_Small
- added C501: 330u, Capacitor_Tantalum_SMD:CP_EIA-7343-31_Kemet-D, symbol zynq_card:C_Polarized
- added C502, C508, C509, C510: 100u, Capacitor_SMD:C_1210_3225Metric, symbol zynq_card:C
- added C503, C504, C516, C517, C518, C522, C523, C524: 4u7, Capacitor_SMD:C_0402_1005Metric, symbol zynq_card:C
- added C505, C506, C507, C513, C514, C515, C519, C520, C521, C525, C526, C527, C529: 470n, Capacitor_SMD:C_0402_1005Metric, symbol zynq_card:C
- added C511, C512: 47u, Capacitor_SMD:C_1210_3225Metric, symbol zynq_card:C
- added C528: 10u, Capacitor_SMD:C_0603_1608Metric, symbol zynq_card:C
- added C61: 47uF, Capacitor_SMD:C_0805_2012Metric, symbol zynq_card:C
- added C67: 100uF, Capacitor_SMD:C_1210_3225Metric, symbol zynq_card:C
- added FB1: 0, Capacitor_SMD:C_0603_1608Metric, symbol zynq_card:R_Small
- added FB501: BLM18SG121TN1D, Inductor_SMD:L_0603_1608Metric, symbol zynq_card:FerriteBead_Small
- added U20: xc7z020clg484, DFTcustom:BGA-484_19.0x19.0mm_Layout22x22_P0.80mm_dia0.40mm, symbol zynq_card:XC7Z020-CLG484
Connections:
- new net 1V0: C11.1, C23.1, C24.1, C28.1, C29.1, C30.1, C31.1, C501.1, C502.1, C503.1, C504.1, C505.1, C506.1, C507.1, C8.1, C9.1, U20.G8 (VCCPINT[6]), U20.H11 (VCCBRAM[2]), U20.H9 (VCCPINT[6]), U20.J10 (VCCBRAM[2]), U20.J12 (VCCINT[8]), U20.J14 (VCCINT[8]), U20.J8 (VCCPINT[6]), U20.K13 (VCCINT[8]), U20.L14 (VCCINT[8]), U20.L8 (VCCPINT[6]), U20.M13 (VCCINT[8]), U20.N14 (VCCINT[8]), U20.N8 (VCCPINT[6]), U20.P13 (VCCINT[8]), U20.R14 (VCCINT[8]), U20.R8 (VCCPINT[6])
- new net 1V35: C513.1, C514.1, C515.1
- new net 1V8: C122.1, C14.1, C15.1, C17.1, C18.1, C19.1, C20.1, C26.1, C4.1, C5.1, C508.1, C509.1, C510.1, C511.1, C512.1, C59.1, FB1.2, FB501.1, U20.K9 (VCCPAUX[4]), U20.M9 (VCCPAUX[4]), U20.P9 (VCCPAUX[4]), U20.T9 (VCCPAUX[4])
- new net 3V3: C114.1, C116.1, C117.1, C118.1, C119.1, C121.1, C46.1, C47.1, C50.1, C516.1, C517.1, C518.1, C519.1, C520.1, C521.1, C522.1, C523.1, C524.1, C525.1, C526.1, C527.1, C55.1, C57.1, C61.1, C65.1, C67.1
- new net GND: C11.2, C114.2, C116.2, C117.2, C118.2, C119.2, C121.2, C122.2, C14.2, C15.2, C17.2, C18.2, C19.2, C20.2, C23.2, C24.2, C26.2, C28.2, C29.2, C30.2, C31.2, C33.2, C34.2, C4.2, C46.2, C47.2, C5.2, C50.2, C501.2, C502.2, C503.2, C504.2, C505.2, C506.2, C507.2, C508.2, C509.2, C510.2, C511.2, C512.2, C513.2, C514.2, C515.2, C516.2, C517.2, C518.2, C519.2, C520.2, C521.2, C522.2, C523.2, C524.2, C525.2, C526.2, C527.2, C528.2, C529.2, C55.2, C57.2, C59.2, C61.2, C65.2, C67.2, C8.2, C9.2, U20.A15 (GND[63]), U20.A5 (GND[63]), U20.AA15 (GND[63]), U20.AA5 (GND[63]), U20.AB18 (GND[63]), U20.AB8 (GND[63]), U20.B18 (GND[63]), U20.B8 (GND[63]), U20.C1 (GND[63]), U20.C11 (GND[63]), U20.C21 (GND[63]), U20.D14 (GND[63]), U20.D4 (GND[63]), U20.E17 (GND[63]), U20.E7 (GND[63]), U20.F10 (GND[63]), U20.F20 (GND[63]), U20.G3 (GND[63]), U20.H12 (GND[63]), U20.H14 (GND[63]), U20.H16 (GND[63]), U20.H6 (GND[63]), U20.H8 (GND[63]), U20.J11 (GND[63]), U20.J13 (GND[63]), U20.J19 (GND[63]), U20.J9 (GND[63]), U20.K10 (GND[63]), U20.K14 (GND[63]), U20.K2 (GND[63]), U20.K22 (GND[63]), U20.K8 (GND[63]), U20.L13 (GND[63]), U20.L15 (GND[63]), U20.L5 (GND[63]), U20.L9 (GND[63]), U20.M10 (GND[63]), U20.M14 (GND[63]), U20.M18 (GND[63]), U20.M8 (GND[63]), U20.N1 (GND[63]), U20.N13 (GND[63]), U20.N21 (GND[63]), U20.N9 (GND[63]), U20.P10 (GND[63]), U20.P12 (GND[63]), U20.P14 (GND[63]), U20.P4 (GND[63]), U20.P8 (GND[63]), U20.R11 (GND[63]), U20.R13 (GND[63]), U20.R17 (GND[63]), U20.R9 (GND[63]), U20.T20 (GND[63]), U20.U13 (GND[63]), U20.U3 (GND[63]), U20.V16 (GND[63]), U20.V6 (GND[63]), U20.W19 (GND[63]), U20.W9 (GND[63]), U20.Y12 (GND[63]), U20.Y2 (GND[63]), U20.Y22 (GND[63])
- new net VCCAUX: C33.1, C34.1, FB1.1, U20.L10 (VCCAUX[4]), U20.N10 (VCCAUX[4]), U20.P11 (VCCAUX[4]), U20.R10 (VCCAUX[4])
- new net VCCPLL: C528.1, C529.1, FB501.2, U20.H10 (VCCPLL)
Other:
- note added: "1V0: VCCINT/VCCBRAM/VCCPINT bulk and the missing mid/high-frequency caps"
- note added: "1V35 VCCO_DDR: 3 more 470n at bank 502"
- note added: "1V8: VCCPAUX, MIO0, MIO1 100u; VCCAUX, VCCO_0 47u"
- note added: "3V3 VCCO_34 (no caps in the block)"
- note added: "3V3 VCCO_35 (no caps in the block)"
- note added: "Block 3V3 caps under U20 (juliancoy's other sheets, source refs): banks 13/33"
- note added: "Block, E6: MIO1 (E12), MIO0 (C6)"
- note added: "E5: VCCPLL from 1V8 through a 120R bead (UG933 Fig. 5-2: BLM18SG121TN1D, GRM188R60J106ME47, GRM155R60J474KE19). Planelet >= 2 mm wide, < 76 mm long, C528 to the H10 via; C529 within 5.1 mm of trace from the H10/GND vias. Replaces juliancoy's direct +1V8."
- note added: "U20 unit 9 and the SoC decoupling. Left/bottom: juliancoy/zynqPCB power.sch (MIT, NOTICE), converted by tools/sheets/05_soc_power.py: only the decaps in the block copper, source refs and positions. Do not edit by hand. Changes: REUSE_LOG.md E5 (VCCPLL through FB501, FB1 = 0 ohm), E6 (C59/C122 on 1V8: MIO banks at 1.8 V). UG933 Tables 3-1/3-2 (CLG484, Z-7020) per merged rail; the C5xx rows add wha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"
- note added: "UG933 count, block + C5xx: 1V0 (VCCINT+VCCBRAM+VCCPINT): 330u 1, 100u 2, 4u7 4, 470n 8 block C28 100u, C9 C24 4u7, C8 C23 C29 C30 C31 470n (+ C11 10u) 1V8 (VCCAUX+VCCPAUX+MIO0+MIO1+VCCO_0): 100u 3, 47u 2, 4u7 4, 470n 5 block C5 C19 C20 C59 C122 4u7, C4 C14 C15 C17 C18 C34 470n (+ C26 C33 10u) VCCPLL: 120R bead + 10u 0603 + 0.47-4.7u 0402 within 5.1 mm of the H10/GND vias 1V35 (VCCO_DDR): 100u 1, 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"

Commit message: LCSC numbers for every BOM part (tools/set_lcsc.py); FB1 as 0 R; U20 = XC7Z020-2CLG484I
tools/set_lcsc.py (run by build_schematic.sh) writes the LCSC field by BOM line: JLC basic parts where there is one,
juliancoy's Murata/Yageo passives bought as basic equivalents (REUSE_LOG E11). FB1, the E5 0 R jumper, gets
0603WAF0000T5E / C21189 (its MPN still named the bead). U20: -2 or -3 speed, any temperature grade (user):
XC7Z020-2CLG484I, C157624. Connectors J1/J2/J3/J5/J6/J9 hand-soldered (no LCSC, skipped in the JLC files).
ERC unchanged (4 intended pin_to_pin), block netlist 0 failures, board rebuilt: parity 0, block copper 0 failures.

Co-Authored-By: Claude Opus 5.5 <noreply@anthropic.com>
Parts:
- C11, C26, C33: LCSC (none) -> C19702; MFR Murata -> (none); MPN GRM188R61A106KE69J -> CL10A106KP8NNNC; SPN 490-14372-1-ND -> (none); SPR Digikey -> (none)
- C114, C122, C503, C504, C516, C517, C518, C522, C523, C524, C57, C59: LCSC (none) -> C23733
- C116, C117, C118, C119, C121, C46, C47, C50, C505, C506, C507, C513, C514, C515, C519, C520, C521, C525, C526, C527, C529, C55, C65: LCSC (none) -> C47339
- C14, C15, C17, C18, C23, C29, C30, C31, C34, C4, C8: LCSC (none) -> C47339; MFR Yageo -> (none); MPN CC0402KRX5R5BB474 -> CL05A474KP5NNNC; SPN 311-1684-1-ND -> (none); SPR Digikey -> (none)
- C19, C20, C24, C5, C9: LCSC (none) -> C23733; MFR Murata -> (none); MPN GRM155R60G475ME47D -> CL05A475MP5NRNC; SPN 490-11980-1-ND -> (none); SPR Digikey -> (none)
- C28: LCSC (none) -> C49066; MFR TAIYO YUDEN -> (none); MPN JMK325ABJ107MM-P -> CL32A107MQVNNNE; SPN 587-4313-1-ND -> (none); SPR Digikey -> (none)
- C501: LCSC (none) -> C116744; MPN (none) -> T520D337M006ATE015
- C502, C508, C509, C510, C67: LCSC (none) -> C49066
- C511, C512: LCSC (none) -> C77101
- C528: LCSC (none) -> C19702
- C61: LCSC (none) -> C16780
- FB1: LCSC (none) -> C21189; MFR Murata Electronics -> UNI-ROYAL; MPN BLM18AG121SN1D -> 0603WAF0000T5E; SPN 490-1011-1-ND -> (none); SPR Digikey -> (none); SPURL - -> (none)
- FB501: LCSC (none) -> C113030
- U20: value xc7z020clg484 -> XC7Z020-2CLG484I; LCSC (none) -> C157624; MPN XC7Z020-1CLG484C -> XC7Z020-2CLG484I
