File: kicad/06_soc_config.kicad_sch (KiCad schematic)
At the start: 0 parts

Commit message: Phase 2: sheet 6 (SoC config): MIO banks, bank 0, boot straps, JTAG
- tools/sheets/06_soc_config.py: U20 units 6/7 (MIO banks 500/501, 1.8 V)
  with every used MIO as a sheet port, boot straps R601-R607 (QSPI boot,
  JTAG cascaded, PLLs on, VMODE 1.8/1.8), PS_POR_B/PS_SRST_B pull-ups,
  PS_MIO_VREF divider; unit 1 (bank 0 at 1.8 V) tied off as on juliancoy,
  R9/R10 kept as block parts, DONE 330R, RSVDGND open (E8)
- J1 (1x5, 3.3 V for FTDI mini-modules) through U601 SN74AVC4T774RSVR,
  the Agilex 3 card's JTAG shifter circuit
- check_block_netlist.py covers sheet 6: on units 1/6/7 only rail/GND balls
  and balls on block-part nets are compared; E3/E7/E8 expected differences;
  J-refs are never block parts (101 parts, 583 pads, 0 failures)
- gen_symbols: SN74AVC4T774 (RSV) box, Conn_01x05; _common: attach(side=),
  pull_r(top=)
- REUSE_LOG E8 and E5/E6 commit refs; ZYNQ_PCB_NOTES JTAG/RSVDGND and the
  UART translator note (needs per-bit direction); STATUS updated

Co-Authored-By: Claude Opus 5.5 <noreply@anthropic.com>
Parts:
- added C601: 10n, Capacitor_SMD:C_0402_1005Metric, symbol zynq_card:C
- added C602, C603: 100n, Capacitor_SMD:C_0402_1005Metric, symbol zynq_card:C
- added J1: JTAG 3V3, Connector_PinHeader_2.54mm:PinHeader_1x05_P2.54mm_Vertical, symbol zynq_card:Conn_01x05
- added R10, R9: 4.7k, Resistor_SMD:R_0402_1005Metric, symbol zynq_card:R
- added R601, R602, R603, R604, R605, R606, R607: 20k, Resistor_SMD:R_0402_1005Metric, symbol zynq_card:R
- added R608, R609, R610, R611, R614, R615, R616: 10k, Resistor_SMD:R_0402_1005Metric, symbol zynq_card:R
- added R612: 330, Resistor_SMD:R_0402_1005Metric, symbol zynq_card:R
- added R613: 1k, Resistor_SMD:R_0402_1005Metric, symbol zynq_card:R
- added U20: XC7Z020-1CLG484I, symbol zynq_card:XC7Z020-CLG484
- added U601: SN74AVC4T774RSVR, Package_DFN_QFN:UQFN-16_1.8x2.6mm_P0.4mm, symbol zynq_card:SN74AVC4T774
Connections:
- new net 1V8: C603.1, R10.2, R604.1, R606.1, R607.1, R608.1, R609.1, R611.1, R612.1, R616.1, R9.2, U20.A10 (VCCO_MIO1_501[4]), U20.B13 (VCCO_MIO1_501[4]), U20.B3 (VCCO_MIO0_500[2]), U20.C6 (VCCO_MIO0_500[2]), U20.D9 (VCCO_MIO1_501[4]), U20.E12 (VCCO_MIO1_501[4]), U20.K11 (VCCADC_0), U20.R12 (VCCO_0), U20.T10 (RSVDVCC3), U20.T7 (RSVDVCC1), U20.T8 (RSVDVCC2), U601.13 (VCCB)
- new net 3V3: C602.1, R614.1, R615.1, U601.14 (VCCA), U601.15 (DIR1), U601.16 (DIR2), U601.5 (DIR3)
- new net GND: C601.2, C602.2, C603.2, J1.5 (Pin_5), R601.2, R602.2, R603.2, R605.2, R610.2, R613.2, U20.G9 (VCCBATT_0), U20.K12 (GNDADC_0), U20.L11 (VP_0), U20.L12 (VREFN_0), U20.M11 (VREFP_0), U20.M12 (VN_0), U20.N11 (DXP_0), U20.N12 (DXN_0), U20.T13 (CFGBVS_0), U601.6 (DIR4), U601.7 (~{OE}), U601.8 (GND)
- new net cfg_done: R612.2, U20.T12 (DONE_0)
- new net cfg_init_n: R10.1, U20.T14 (INIT_B_0)
- new net cfg_program_n: R9.1, U20.T11 (PROGRAM_B_0)
- new net emmc_rst_n: R606.2, U20.D5 (PS_MIO7_500)
- new net eth_int_n: U20.G7 (PS_MIO10_500)
- new net eth_rst_n: U20.C4 (PS_MIO9_500)
- new net i2c_scl: U20.D13 (PS_MIO50_501)
- new net i2c_sda: U20.C10 (PS_MIO51_501)
- new net jtag_tck: J1.2 (Pin_2), R613.1, U601.1 (A1)
- new net jtag_tck_1v8: U20.G11 (TCK_0), U601.12 (B1)
- new net jtag_tdi: J1.1 (Pin_1), R615.2, U601.2 (A2)
- new net jtag_tdi_1v8: U20.H13 (TDI_0), U601.11 (B2)
- new net jtag_tdo: J1.4 (Pin_4), U601.4 (A4)
- new net jtag_tdo_1v8: R616.2, U20.G14 (TDO_0), U601.9 (B4)
- new net jtag_tms: J1.3 (Pin_3), R614.2, U601.3 (A3)
- new net jtag_tms_1v8: U20.G12 (TMS_0), U601.10 (B3)
- new net mdc: U20.D10 (PS_MIO52_501)
- new net mdio: U20.C12 (PS_MIO53_501)
- new net ps_clk: U20.F7 (PS_CLK_500)
- new net ps_mio_vref: C601.1, R609.2, R610.1, U20.F8 (PS_MIO_VREF_501)
- new net ps_por_n: R608.2, U20.B5 (PS_POR_B_500)
- new net ps_srst_n: R611.2, U20.C9 (PS_SRST_B_501)
- new net qspi_cs_n: U20.A1 (PS_MIO1_500)
- new net qspi_fbclk: R607.2, U20.E5 (PS_MIO8_500)
- new net qspi_io0: R601.1, U20.A2 (PS_MIO2_500)
- new net qspi_io1: R602.1, U20.F6 (PS_MIO3_500)
- new net qspi_io2: R603.1, U20.E4 (PS_MIO4_500)
- new net qspi_io3: R604.2, U20.A3 (PS_MIO5_500)
- new net qspi_sclk: R605.1, U20.A4 (PS_MIO6_500)
- new net rgmii_rx_ctl: U20.D7 (PS_MIO27_501)
- new net rgmii_rxc: U20.A14 (PS_MIO22_501)
- new net rgmii_rxd0: U20.E11 (PS_MIO23_501)
- new net rgmii_rxd1: U20.B7 (PS_MIO24_501)
- new net rgmii_rxd2: U20.F12 (PS_MIO25_501)
- new net rgmii_rxd3: U20.A13 (PS_MIO26_501)
- new net rgmii_tx_ctl: U20.F11 (PS_MIO21_501)
- new net rgmii_txc: U20.D6 (PS_MIO16_501)
- new net rgmii_txd0: U20.E9 (PS_MIO17_501)
- new net rgmii_txd1: U20.A7 (PS_MIO18_501)
- new net rgmii_txd2: U20.E10 (PS_MIO19_501)
- new net rgmii_txd3: U20.A8 (PS_MIO20_501)
- new net sd_clk: U20.E14 (PS_MIO40_501)
- new net sd_cmd: U20.C8 (PS_MIO41_501)
- new net sd_dat0: U20.D8 (PS_MIO42_501)
- new net sd_dat1: U20.B11 (PS_MIO43_501)
- new net sd_dat2: U20.E13 (PS_MIO44_501)
- new net sd_dat3: U20.B9 (PS_MIO45_501)
- new net uart_rx: U20.C14 (PS_MIO49_501)
- new net uart_tx: U20.D11 (PS_MIO48_501)
- no-connect marks 0 -> 21
Other:
- note added: "Boot straps (sampled at PS_POR_B release), 20 k each, pull-ups to VCCO_MIO0 (1V8): MIO2 = 0 JTAG cascaded, MIO5/4/3 = 1/0/0 QSPI boot, MIO6 = 0 PLLs on, MIO7 = 1 / MIO8 = 1: banks 500/501 at 1.8 V (must match VCCO_MIO0/1). PS_POR_B: open drain from the supervisor (sheet 4), 10 k up."
- note added: "CFGBVS to GND: bank 0 at 1.8 V. XADC unused: VCCADC 1V8, analog inputs to GND. RSVDGND open (UG865 v1.9; REUSE_LOG E8). RSVDVCC to VCCO_0."
- note added: "J1: 1 TDI, 2 TCK, 3 TMS, 4 TDO, 5 GND (family pinout)"
- note added: "JTAG pulls: TCK 1 k down, TMS/TDI 10 k up (3.3 V side); 10 k up on TDO at 1.8 V (B4 defined while TDO is off)."
- note added: "JTAG: J1 at 3.3 V (FTDI mini-module, no VREF), U601 SN74AVC4T774RSVR (C779392) to bank 0 at 1.8 V, as on the Agilex 3 card. DIR1-3 = H: TCK/TDI/TMS A->B; DIR4 = L: TDO B->A; OE low."
- note added: "MIO0, MIO11-15: spare"
- note added: "MIO28-39 (USB0), 46, 47: spare"
- note added: "PROGRAM_B / INIT_B: juliancoy's R9/R10 (block), 4.7 k to VCCO_0. DONE: 330 R to VCCO_0 [verify UG470]."
- note added: "PS MIO banks 500/501 (1.8 V) and bank 0 (configuration, 1.8 V as on juliancoy). Pin plan: vivado/pinplan/mio.csv; rules: ZYNQ_PCB_NOTES.md §4-5, §7. Interfaces leave as sheet ports; their pull-ups sit with the parts on their sheets. JTAG J1 is 3.3 V (FTDI mini-module), shifted by U601."
- note added: "PS_MIO_VREF = 0.9 V (HSTL 1.8 V RGMII receivers): 10 k / 10 k + 10 n. PS_SRST_B: 10 k to VCCO_MIO1; must stay high while the BootROM runs (no button)."

Commit message: LCSC numbers for every BOM part (tools/set_lcsc.py); FB1 as 0 R; U20 = XC7Z020-2CLG484I
tools/set_lcsc.py (run by build_schematic.sh) writes the LCSC field by BOM line: JLC basic parts where there is one,
juliancoy's Murata/Yageo passives bought as basic equivalents (REUSE_LOG E11). FB1, the E5 0 R jumper, gets
0603WAF0000T5E / C21189 (its MPN still named the bead). U20: -2 or -3 speed, any temperature grade (user):
XC7Z020-2CLG484I, C157624. Connectors J1/J2/J3/J5/J6/J9 hand-soldered (no LCSC, skipped in the JLC files).
ERC unchanged (4 intended pin_to_pin), block netlist 0 failures, board rebuilt: parity 0, block copper 0 failures.

Co-Authored-By: Claude Opus 5.5 <noreply@anthropic.com>
Parts:
- C601: LCSC (none) -> C15195
- C602, C603: LCSC (none) -> C1525
- R10, R9: LCSC (none) -> C25900
- R601, R602, R603, R604, R605, R606, R607: LCSC (none) -> C25765
- R608, R609, R610, R611, R614, R615, R616: LCSC (none) -> C25744
- R612: LCSC (none) -> C25104
- R613: LCSC (none) -> C11702
- U20: value XC7Z020-1CLG484I -> XC7Z020-2CLG484I
Changed lines of the file:
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@@
 			)
 		)
-		(property "Value" "XC7Z020-1CLG484I"
+		(property "Value" "XC7Z020-2CLG484I"
 			(at 91.44 34.29 0)
 			(effects
@@
 			)
 		)
+		(property "LCSC" "C25765"
+			(at 17.78 132.08 0)
+			(effects
+				(font
+					(size 1.27 1.27)
+				)
+				(hide yes)
+			)
+		)
 		(property "Description" "Resistor"
 			(at 17.78 132.08 0)
@@
 			)
 		)
+		(property "LCSC" "C25765"
+			(at 29.21 132.08 0)
+			(effects
+				(font
+					(size 1.27 1.27)
+				)
+				(hide yes)
+			)
+		)
 		(property "Description" "Resistor"
 			(at 29.21 132.08 0)
@@
 			)
 		)
+		(property "LCSC" "C25765"
+			(at 40.64 132.08 0)
+			(effects
+				(font
+					(size 1.27 1.27)
+				)
+				(hide yes)
+			)
+		)
 		(property "Description" "Resistor"
 			(at 40.64 132.08 0)
@@
 			)
 		)
+		(property "LCSC" "C25765"
+			(at 52.07 132.08 0)
+			(effects
+				(font
+					(size 1.27 1.27)
+				)
+				(hide yes)
+			)
+		)
 		(property "Description" "Resistor"
 			(at 52.07 132.08 0)
@@
 			)
 		)
+		(property "LCSC" "C25765"
+			(at 63.5 132.08 0)
+			(effects
+				(font
+					(size 1.27 1.27)
+				)
+				(hide yes)
+			)
+		)
 		(property "Description" "Resistor"
 			(at 63.5 132.08 0)
@@
 			)
 		)
+		(property "LCSC" "C25765"
+			(at 74.93 132.08 0)
+			(effects
+				(font
+					(size 1.27 1.27)
+				)
+				(hide yes)
+			)
+		)
 		(property "Description" "Resistor"
 			(at 74.93 132.08 0)
@@
 			)
 		)
+		(property "LCSC" "C25765"
+			(at 86.36 132.08 0)
+			(effects
+				(font
+					(size 1.27 1.27)
+				)
+				(hide yes)
+			)
+		)
 		(property "Description" "Resistor"
 			(at 86.36 132.08 0)
@@
 			)
 		)
+		(property "LCSC" "C25744"
+			(at 97.79 132.08 0)
+			(effects
+				(font
+					(size 1.27 1.27)
+				)
+				(hide yes)
+			)
+		)
 		(property "Description" "Resistor"
 			(at 97.79 132.08 0)
@@
 			)
 		)
-		(property "Value" "XC7Z020-1CLG484I"
+		(property "Value" "XC7Z020-2CLG484I"
 			(at 226.06 26.67 0)
 			(effects
@@
 			)
 		)
+		(property "LCSC" "C25744"
+			(at 139.7 177.8 0)
+			(effects
+				(font
+					(size 1.27 1.27)
+				)
+				(hide yes)
+			)
+		)
 		(property "Description" "Resistor"
 			(at 139.7 177.8 0)
@@
 			)
 		)
+		(property "LCSC" "C25744"
+			(at 151.13 177.8 0)
+			(effects
+				(font
+					(size 1.27 1.27)
+				)
+				(hide yes)
+			)
+		)
 		(property "Description" "Resistor"
 			(at 151.13 177.8 0)
@@
 			)
 		)
+		(property "LCSC" "C15195"
+			(at 162.56 177.8 0)
+			(effects
+				(font
+					(size 1.27 1.27)
+				)
+				(hide yes)
+			)
+		)
 		(property "Description" "Unpolarized capacitor"
 			(at 162.56 177.8 0)
@@
 			)
 		)
+		(property "LCSC" "C25744"
+			(at 182.88 177.8 0)
+			(effects
+				(font
+					(size 1.27 1.27)
+				)
+				(hide yes)
+			)
+		)
 		(property "Description" "Resistor"
 			(at 182.88 177.8 0)
@@
 			)
 		)
-		(property "Value" "XC7Z020-1CLG484I"
+		(property "Value" "XC7Z020-2CLG484I"
 			(at 368.3 34.29 0)
 			(effects
@@
 			)
 		)
+		(property "LCSC" "C25900"
+			(at 294.64 132.08 0)
+			(effects
+				(font
+					(size 1.27 1.27)
+				)
+				(hide yes)
+			)
+		)
 		(property "Description" "Resistor"
 			(at 294.64 132.08 0)
@@
 			)
 		)
+		(property "LCSC" "C25900"
+			(at 306.07 132.08 0)
+			(effects
+				(font
+					(size 1.27 1.27)
+				)
+				(hide yes)
+			)
+		)
 		(property "Description" "Resistor"
 			(at 306.07 132.08 0)
@@
 			)
 		)
+		(property "LCSC" "C25104"
+			(at 317.5 132.08 0)
+			(effects
+				(font
+					(size 1.27 1.27)
+				)
+				(hide yes)
+			)
+		)
 		(property "Description" "Resistor"
 			(at 317.5 132.08 0)
@@
 			)
 		)
+		(property "LCSC" "C1525"
+			(at 309.88 220.98 0)
+			(effects
+				(font
+					(size 1.27 1.27)
+				)
+				(hide yes)
+			)
+		)
 		(property "Description" "Unpolarized capacitor"
 			(at 309.88 220.98 0)
@@
 			)
 		)
+		(property "LCSC" "C1525"
+			(at 353.06 220.98 0)
+			(effects
+				(font
+					(size 1.27 1.27)
+				)
+				(hide yes)
+			)
+		)
 		(property "Description" "Unpolarized capacitor"
 			(at 353.06 220.98 0)
@@
 			)
 		)
+		(property "LCSC" "C11702"
+			(at 226.06 233.68 0)
+			(effects
+				(font
+					(size 1.27 1.27)
+				)
+				(hide yes)
+			)
+		)
 		(property "Description" "Resistor"
 			(at 226.06 233.68 0)
@@
 			)
 		)
+		(property "LCSC" "C25744"
+			(at 237.49 233.68 0)
+			(effects
+				(font
+					(size 1.27 1.27)
+				)
+				(hide yes)
+			)
+		)
 		(property "Description" "Resistor"
 			(at 237.49 233.68 0)
@@
 			)
 		)
+		(property "LCSC" "C25744"
+			(at 248.92 233.68 0)
+			(effects
+				(font
+					(size 1.27 1.27)
+				)
+				(hide yes)
+			)
+		)
 		(property "Description" "Resistor"
 			(at 248.92 233.68 0)
@@
 			(at 260.35 233.68 0)
 			(effects
+				(font
+					(size 1.27 1.27)
+				)
+				(hide yes)
+			)
+		)
+		(property "LCSC" "C25744"
+			(at 260.35 233.68 0)
+			(effects
