File: kicad/07_clocks.kicad_sch (KiCad schematic)
At the start: 0 parts

Commit message: Phase 2: sheet 7 (clocks): 33.333 MHz PS_CLK oscillator
- tools/sheets/07_clocks.py: Y701 YXC OT322533.3333MJBA4SL (C2831392,
  1.8 V CMOS, 3225) with the Agilex 3 card's oscillator circuit: EN tied
  to VDD, FB701 BLM18PG121SN1D + C701 470n supply filter, R701 33R
  source-series to the ps_clk port (U20 F7)
- gen_symbols: Oscillator:ASE-xxxMHz
- STATUS updated; REUSE_LOG E8 commit ref

Co-Authored-By: Claude Opus 5.5 <noreply@anthropic.com>
Parts:
- added C701: 470n, Capacitor_SMD:C_0402_1005Metric, symbol zynq_card:C
- added FB701: BLM18PG121SN1D, Inductor_SMD:L_0603_1608Metric, symbol zynq_card:FerriteBead_Small
- added R701: 33, Resistor_SMD:R_0402_1005Metric, symbol zynq_card:R
- added Y701: 33.333MHz, Oscillator:Oscillator_SMD_Abracon_ASE-4Pin_3.2x2.5mm, symbol zynq_card:ASE-xxxMHz
Connections:
- new net: R701.1, Y701.3 (OUT)
- new net 1V8: FB701.1
- new net GND: C701.2, Y701.2 (GND)
- new net osc_vdd: C701.1, FB701.2, Y701.1 (EN), Y701.4 (Vdd)
- new net ps_clk: R701.2
Other:
- note added: "PS_CLK: Y701 33.333 MHz, 1.8 V CMOS (bank 500 = VCCO_MIO0 = 1.8 V) -> R701 33 R at Y701 -> ps_clk (U20 F7). Circuit of the Agilex 3 card's oscillator: EN tied to VDD, supply through FB701 with C701 470 n. Layout: Y701 close to F7, one point-to-point trace, R701 at the oscillator pin."

Commit message: LCSC numbers for every BOM part (tools/set_lcsc.py); FB1 as 0 R; U20 = XC7Z020-2CLG484I
tools/set_lcsc.py (run by build_schematic.sh) writes the LCSC field by BOM line: JLC basic parts where there is one,
juliancoy's Murata/Yageo passives bought as basic equivalents (REUSE_LOG E11). FB1, the E5 0 R jumper, gets
0603WAF0000T5E / C21189 (its MPN still named the bead). U20: -2 or -3 speed, any temperature grade (user):
XC7Z020-2CLG484I, C157624. Connectors J1/J2/J3/J5/J6/J9 hand-soldered (no LCSC, skipped in the JLC files).
ERC unchanged (4 intended pin_to_pin), block netlist 0 failures, board rebuilt: parity 0, block copper 0 failures.

Co-Authored-By: Claude Opus 5.5 <noreply@anthropic.com>
Parts:
- C701: LCSC (none) -> C47339
- R701: LCSC (none) -> C25105
Changed lines of the file:
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@@
+			)
+		)
+		(property "LCSC" "C47339"
+			(at 60.96 68.58 0)
+			(effects
+				(font
+					(size 1.27 1.27)
+				)
+				(hide yes)
 			)
 		)
@@
 			(at 109.22 63.5 0)
 			(effects
+				(font
+					(size 1.27 1.27)
+				)
+				(hide yes)
+			)
+		)
+		(property "LCSC" "C25105"
+			(at 109.22 63.5 0)
+			(effects
