File: kicad/08_qspi.kicad_sch (KiCad schematic)
At the start: 0 parts

Commit message: Phase 2: sheets 8-10 (QSPI flash, RTL8211F Ethernet, eMMC)
Sheet 8: IS25WP128-RHLE on QSPI0 at 1V8, CS# pull-up, RESET# on ps_por_n.
Sheet 9: the Ti135 RTL8211FDI-CG + HR911130A sheet on GEM0 RGMII / MDIO0.
RGMII and MDIO pads at 1.8 V via the PHY's internal LDO; INTB is open drain,
so its 1V8 pull-up is fine (closes the INTB [verify]). eth_rst_n pull-down
is 1k to beat the MIO reset pull-up.
Sheet 10: THGAMVG7T13BAIL on SD0, 4-bit, with the KIOXIA decoupling values.
Symbols ported from the Ti135 card into gen_symbols.py; its flash and RJ45
footprints copied into lib/zynq_card.pretty. fill_footprints() in _common.py.
Every port checked against the U20 MIO balls in the netlist. ERC: only the
UART/I2C ports and the PL bank units remain; block check 0 failures.

Co-Authored-By: Claude Opus 5.5 <noreply@anthropic.com>
Parts:
- added C801: 100n, Capacitor_SMD:C_0402_1005Metric, symbol zynq_card:C
- added R801: 10k, Resistor_SMD:R_0402_1005Metric, symbol zynq_card:R
- added U801: IS25WP128-RHLE, zynq_card:MX25U25645G_CSP24_6x8mm_P1.0mm, symbol zynq_card:IS25WP128-RHLE
Connections:
- new net 1V8: C801.1, R801.1, U801.B4 (VCC)
- new net GND: C801.2, U801.B3 (GND)
- new net ps_por_n: U801.A4 (RESET#)
- new net qspi_cs_n: R801.2, U801.C2 (CS#)
- new net qspi_io0: U801.D3 (SI/IO0)
- new net qspi_io1: U801.D2 (SO/IO1)
- new net qspi_io2: U801.C4 (WP#/IO2)
- new net qspi_io3: U801.D4 (HOLD#/IO3)
- new net qspi_sclk: U801.B2 (SCLK)
Other:
- note added: "QSPI boot flash (ZYNQ_PCB_NOTES.md §4.3): U801 IS25WP128-RHLE, 1.8 V, on QSPI0 = MIO1-6 (bank 500). Boot straps on IO0-3/SCLK are on sheet 6 (20 k). CS# pull-up R801; RESET# on ps_por_n (supervisor, sheet 4). Layout (UG933 QSPI): IO0-3 and CS# matched to SCLK within +/-50 ps; MIO8 (feedback clock) stays a short stub."
- note added: "R801: CS# high while MIO1 is tri-stated"
- note added: "U801 VCC (B4)"

Commit message: LCSC numbers for every BOM part (tools/set_lcsc.py); FB1 as 0 R; U20 = XC7Z020-2CLG484I
tools/set_lcsc.py (run by build_schematic.sh) writes the LCSC field by BOM line: JLC basic parts where there is one,
juliancoy's Murata/Yageo passives bought as basic equivalents (REUSE_LOG E11). FB1, the E5 0 R jumper, gets
0603WAF0000T5E / C21189 (its MPN still named the bead). U20: -2 or -3 speed, any temperature grade (user):
XC7Z020-2CLG484I, C157624. Connectors J1/J2/J3/J5/J6/J9 hand-soldered (no LCSC, skipped in the JLC files).
ERC unchanged (4 intended pin_to_pin), block netlist 0 failures, board rebuilt: parity 0, block copper 0 failures.

Co-Authored-By: Claude Opus 5.5 <noreply@anthropic.com>
Parts:
- C801: LCSC (none) -> C1525
- R801: LCSC (none) -> C25744
Changed lines of the file:
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@@
+			)
+		)
+		(property "LCSC" "C25744"
+			(at 86.36 104.14 0)
+			(effects
+				(font
+					(size 1.27 1.27)
+				)
+				(hide yes)
 			)
 		)
@@
 			(at 147.32 106.68 0)
 			(effects
+				(font
+					(size 1.27 1.27)
+				)
+				(hide yes)
+			)
+		)
+		(property "LCSC" "C1525"
+			(at 147.32 106.68 0)
+			(effects
