File: kicad/09_ethernet.kicad_sch (KiCad schematic)
At the start: 0 parts

Commit message: Phase 2: sheets 8-10 (QSPI flash, RTL8211F Ethernet, eMMC)
Sheet 8: IS25WP128-RHLE on QSPI0 at 1V8, CS# pull-up, RESET# on ps_por_n.
Sheet 9: the Ti135 RTL8211FDI-CG + HR911130A sheet on GEM0 RGMII / MDIO0.
RGMII and MDIO pads at 1.8 V via the PHY's internal LDO; INTB is open drain,
so its 1V8 pull-up is fine (closes the INTB [verify]). eth_rst_n pull-down
is 1k to beat the MIO reset pull-up.
Sheet 10: THGAMVG7T13BAIL on SD0, 4-bit, with the KIOXIA decoupling values.
Symbols ported from the Ti135 card into gen_symbols.py; its flash and RJ45
footprints copied into lib/zynq_card.pretty. fill_footprints() in _common.py.
Every port checked against the U20 MIO balls in the netlist. ERC: only the
UART/I2C ports and the PL bank units remain; block check 0 failures.

Co-Authored-By: Claude Opus 5.5 <noreply@anthropic.com>
Parts:
- added C901, C921, C922, C931, C932, C933, C934, C936, C941, C950, C951: 100n, Capacitor_SMD:C_0402_1005Metric, symbol zynq_card:C
- added C910, C911: 27p, Capacitor_SMD:C_0402_1005Metric, symbol zynq_card:C
- added C920: 10u, Capacitor_SMD:C_0805_2012Metric, symbol zynq_card:C
- added C930, C935, C940: 1u, Capacitor_SMD:C_0402_1005Metric, symbol zynq_card:C
- added FB901: BLM15PX121SN1D, Inductor_SMD:L_0402_1005Metric, symbol zynq_card:FerriteBead_Small
- added J9: HR911130A, zynq_card:RJ45_Hanrun_HR911130A_Horizontal, symbol zynq_card:HR911130A
- added R901, R902, R903, R904, R905, R906, R907, R908, R909, R910, R911, R912: 22R, Resistor_SMD:R_0402_1005Metric, symbol zynq_card:R
- added R920, R921, R922, R923, R924, R925, R926, R927, R928, R929, R930: 4k7, Resistor_SMD:R_0402_1005Metric, symbol zynq_card:R
- added R931: 2.49k 1%, Resistor_SMD:R_0402_1005Metric, symbol zynq_card:R
- added R932: 10k, Resistor_SMD:R_0402_1005Metric, symbol zynq_card:R
- added R933: 1k, Resistor_SMD:R_0402_1005Metric, symbol zynq_card:R
- added R950: 330R, Resistor_SMD:R_0402_1005Metric, symbol zynq_card:R
- added U901: RTL8211FDI-CG, Package_DFN_QFN:QFN-40-1EP_5x5mm_P0.4mm_EP3.6x3.6mm_ThermalVias, symbol zynq_card:RTL8211FD
- added U902: 74LVC1G07GW, Package_TO_SOT_SMD:SOT-353_SC-70-5, symbol zynq_card:74LVC1G07
- added Y901: 25MHz, Crystal:Crystal_SMD_3225-4Pin_3.2x2.5mm, symbol zynq_card:Crystal_GND24
Connections:
- new net 1V8: C951.1, R929.1, R930.1, U902.5 (VCC)
- new net 3V3: C940.1, C941.1, FB901.1, R928.1, R932.1, R950.1, U901.29 (DVDD33)
- new net GND: C901.2, C910.2, C911.2, C920.2, C921.2, C922.2, C930.2, C931.2, C932.2, C933.2, C934.2, C935.2, C936.2, C940.2, C941.2, C950.2, C951.2, J9.10 (CHS), J9.SH (SHIELD), R921.2, R922.2, R923.2, R924.2, R926.2, R927.2, R931.2, R933.2, U901.41 (GND), U902.3 (GND), Y901.2 (G), Y901.4 (G)
- new net eth_ct: C950.1, J9.1 (TCT)
- new net eth_int_n: R930.2, U901.31 (INTB/PMEB)
- new net eth_led_a: J9.11 (LEDG_A), R950.2
- new net eth_led_k: J9.12 (LEDG_K), R928.2, U901.34 (LED2/CFG_LDO1)
- new net eth_mdi_a_N: J9.3 (MDI0-), U901.2 (MDIN0)
- new net eth_mdi_a_P: J9.2 (MDI0+), U901.1 (MDIP0)
- new net eth_mdi_b_N: J9.7 (MDI1-), U901.5 (MDIN1)
- new net eth_mdi_b_P: J9.4 (MDI1+), U901.4 (MDIP1)
- new net eth_mdi_c_N: J9.6 (MDI2-), U901.7 (MDIN2)
- new net eth_mdi_c_P: J9.5 (MDI2+), U901.6 (MDIP2)
- new net eth_mdi_d_N: J9.9 (MDI3-), U901.10 (MDIN3)
- new net eth_mdi_d_P: J9.8 (MDI3+), U901.9 (MDIP3)
- new net eth_rst_n: R933.1, U902.2
- new net mdc: U901.13 (MDC)
- new net mdio: R929.2, U901.14 (MDIO)
- new net phy_avdd33: C920.1, C921.1, C922.1, FB901.2, U901.11 (AVDD33), U901.40 (AVDD33)
- new net phy_dvdd_rg: C935.1, C936.1, R920.1, R925.1, U901.28 (DVDD_RG)
- new net phy_led0: R926.1, U901.32 (LED0/CFG_EXT)
- new net phy_led1: R927.1, U901.33 (LED1/CFG_LDO0)
- new net phy_rset: R931.1, U901.39 (RSET)
- new net phy_rstb: C901.1, R932.2, U901.12 (PHYRSTB), U902.4
- new net phy_rx_ctl: R908.2, R922.1, U901.26 (RXCTL/PHYAD2)
- new net phy_rxc: R907.2, R921.1, U901.27 (RXC/PHYAD1)
- new net phy_rxd0: R909.2, R925.2, U901.25 (RXD0/RXDLY)
- new net phy_rxd1: R910.2, R924.1, U901.24 (RXD1/TXDLY)
- new net phy_rxd2: R911.2, R923.1, U901.23 (RXD2/PLLOFF)
- new net phy_rxd3: R912.2, R920.2, U901.22 (RXD3/PHYAD0)
- new net phy_tx_ctl: R902.2, U901.19 (TXCTL)
- new net phy_txc: R901.2, U901.20 (TXC)
- new net phy_txd0: R903.2, U901.18 (TXD0)
- new net phy_txd1: R904.2, U901.17 (TXD1)
- new net phy_txd2: R905.2, U901.16 (TXD2)
- new net phy_txd3: R906.2, U901.15 (TXD3)
- new net phy_vdd10: C930.1, C931.1, C932.1, C933.1, C934.1, U901.21 (DVDD10), U901.3 (AVDD10), U901.30 (LDO_OUT), U901.38 (AVDD10), U901.8 (AVDD10)
- new net phy_xi: C910.1, U901.36 (XTAL_IN), Y901.1
- new net phy_xo: C911.1, U901.37 (XTAL_OUT), Y901.3
- new net rgmii_rx_ctl: R908.1
- new net rgmii_rxc: R907.1
- new net rgmii_rxd0: R909.1
- new net rgmii_rxd1: R910.1
- new net rgmii_rxd2: R911.1
- new net rgmii_rxd3: R912.1
- new net rgmii_tx_ctl: R902.1
- new net rgmii_txc: R901.1
- new net rgmii_txd0: R903.1
- new net rgmii_txd1: R904.1
- new net rgmii_txd2: R905.1
- new net rgmii_txd3: R906.1
- no-connect marks 0 -> 4
Other:
- note added: "25 MHz crystal 3225, 27 p load (Agilex card values), +/-50 ppm total; place at the PHY"
- note added: "AVDD33 (pins 11, 40) through a ferrite: 10u + 2 x 100n"
- note added: "DVDD33 (pin 29)"
- note added: "DVDD_RG: RGMII pad LDO output (1.8 V), caps only"
- note added: "Jack LED: green anode via R950 to 3V3, cathode on PHY LED2 (3.3 V pin, active low with its CFG_LDO1 pull-up R928). Program LCR for link/activity."
- note added: "LDO_OUT 1.0 V -> AVDD10 (3, 8, 38) + DVDD10 (21) only: 1u + 4 x 100n (>= 0.1u, Table 9.2)"
- note added: "PHYRSTB is a 3.3 V input: U902 74LVC1G07 (1V8 supply) open drain, R932 10k to 3V3, C901 filter. R933 1k holds eth_rst_n (MIO9) low against the MIO reset pull-up until software releases the PHY."
- note added: "RGMII series 22 R: TX at the SoC (MIO), RX at the PHY (source side)"
- note added: "RTL8211FDI-CG gigabit PHY, RGMII at 1.8 V (internal pad LDO) to GEM0 (MIO16-27, bank 501), MDIO0 on MIO52/53, PHY address 1. 3.3 V only: core 1.0 V from its own LDO. J9 = HanRun HR911130A magjack (green LED from LED2, yellow spare), placed per MECHANICAL.md."
- note added: "Straps 4k7: PHYAD = 001 (RXD3 up, RXC/RXCTL down), PLLOFF/TXDLY = 0, RXDLY = 1 (RX pins to DVDD_RG); CFG_EXT = 0 (LED0 down), CFG_LDO = 10 (LED1 down, LED2 up to 3V3) -> 1.8 V RGMII pads. MDIO/INT_N pull-ups to 1V8."

Commit message: LCSC numbers for every BOM part (tools/set_lcsc.py); FB1 as 0 R; U20 = XC7Z020-2CLG484I
tools/set_lcsc.py (run by build_schematic.sh) writes the LCSC field by BOM line: JLC basic parts where there is one,
juliancoy's Murata/Yageo passives bought as basic equivalents (REUSE_LOG E11). FB1, the E5 0 R jumper, gets
0603WAF0000T5E / C21189 (its MPN still named the bead). U20: -2 or -3 speed, any temperature grade (user):
XC7Z020-2CLG484I, C157624. Connectors J1/J2/J3/J5/J6/J9 hand-soldered (no LCSC, skipped in the JLC files).
ERC unchanged (4 intended pin_to_pin), block netlist 0 failures, board rebuilt: parity 0, block copper 0 failures.

Co-Authored-By: Claude Opus 5.5 <noreply@anthropic.com>
Parts:
- C901, C921, C922, C931, C932, C933, C934, C936, C941, C950, C951: LCSC (none) -> C1525
- C910, C911: LCSC (none) -> C107002
- C920: LCSC (none) -> C15850
- C930, C935, C940: LCSC (none) -> C52923
- FB901: LCSC (none) -> C88970
- R901, R902, R903, R904, R905, R906, R907, R908, R909, R910, R911, R912: LCSC (none) -> C25092
- R920, R921, R922, R923, R924, R925, R926, R927, R928, R929, R930: LCSC (none) -> C25900
- R931: LCSC (none) -> C25884
- R932: LCSC (none) -> C25744
- R933: LCSC (none) -> C11702
- R950: LCSC (none) -> C25104
- Y901: LCSC (none) -> C70593; MPN (none) -> X322525MRB4SI
