File: kicad/10_emmc.kicad_sch (KiCad schematic)
At the start: 0 parts

Commit message: Phase 2: sheets 8-10 (QSPI flash, RTL8211F Ethernet, eMMC)
Sheet 8: IS25WP128-RHLE on QSPI0 at 1V8, CS# pull-up, RESET# on ps_por_n.
Sheet 9: the Ti135 RTL8211FDI-CG + HR911130A sheet on GEM0 RGMII / MDIO0.
RGMII and MDIO pads at 1.8 V via the PHY's internal LDO; INTB is open drain,
so its 1V8 pull-up is fine (closes the INTB [verify]). eth_rst_n pull-down
is 1k to beat the MIO reset pull-up.
Sheet 10: THGAMVG7T13BAIL on SD0, 4-bit, with the KIOXIA decoupling values.
Symbols ported from the Ti135 card into gen_symbols.py; its flash and RJ45
footprints copied into lib/zynq_card.pretty. fill_footprints() in _common.py.
Every port checked against the U20 MIO balls in the netlist. ERC: only the
UART/I2C ports and the PL bank units remain; block check 0 failures.

Co-Authored-By: Claude Opus 5.5 <noreply@anthropic.com>
Parts:
- added C1001, C1003: 4u7, Capacitor_SMD:C_0402_1005Metric, symbol zynq_card:C
- added C1002: 220n, Capacitor_SMD:C_0402_1005Metric, symbol zynq_card:C
- added C1004: 100n, Capacitor_SMD:C_0402_1005Metric, symbol zynq_card:C
- added C1005: 2u2, Capacitor_SMD:C_0402_1005Metric, symbol zynq_card:C
- added R1001: 0R, Resistor_SMD:R_0402_1005Metric, symbol zynq_card:R
- added R1010, R1011, R1012, R1013, R1014, R1015, R1016, R1017, R1018, R1019: 47k, Resistor_SMD:R_0402_1005Metric, symbol zynq_card:R
- added U1001: THGAMVG7T13BAIL, Package_BGA:LFBGA-153_11.5x13mm_Layout14x14_P0.5mm, symbol zynq_card:THGAMVG7T13BAIL
Connections:
- new net 1V8: C1003.1, C1004.1, R1010.1, R1011.1, R1012.1, R1013.1, R1014.1, R1015.1, R1016.1, R1017.1, R1018.1, U1001.C6 (VCCQ), U1001.M4 (VCCQ), U1001.N4 (VCCQ), U1001.P3 (VCCQ), U1001.P5 (VCCQ)
- new net 3V3: C1001.1, C1002.1, U1001.E6 (VCC), U1001.F5 (VCC), U1001.J10 (VCC), U1001.K9 (VCC)
- new net GND: C1001.2, C1002.2, C1003.2, C1004.2, C1005.2, R1019.2, U1001.A6 (VSS), U1001.C4 (VSSQ), U1001.E7 (VSS), U1001.G5 (VSS), U1001.H10 (VSS), U1001.J5 (VSS), U1001.K8 (VSS), U1001.N2 (VSSQ), U1001.N5 (VSSQ), U1001.P4 (VSSQ), U1001.P6 (VSSQ)
- new net emmc_clk: R1001.2, U1001.M6 (CLK)
- new net emmc_dat4: R1015.2, U1001.B3 (DAT4)
- new net emmc_dat5: R1016.2, U1001.B4 (DAT5)
- new net emmc_dat6: R1017.2, U1001.B5 (DAT6)
- new net emmc_dat7: R1018.2, U1001.B6 (DAT7)
- new net emmc_ds: R1019.1, U1001.H5 (DS)
- new net emmc_rst_n: U1001.K5 (RST_n)
- new net emmc_vddi: C1005.1, U1001.C2 (VDDi)
- new net sd_clk: R1001.1
- new net sd_cmd: R1010.2, U1001.M5 (CMD)
- new net sd_dat0: R1011.2, U1001.A3 (DAT0)
- new net sd_dat1: R1012.2, U1001.A4 (DAT1)
- new net sd_dat2: R1013.2, U1001.A5 (DAT2)
- new net sd_dat3: R1014.2, U1001.B2 (DAT3)
Other:
- note added: "47 k pull-ups to 1V8 (CMD, DAT0-7; DAT4-7 unused in 4-bit mode); DS (HS400 strobe, unused) 47 k pull-down"
- note added: "R1001: at the MIO40 pin"
- note added: "VCC 3V3: 4u7 + 220n"
- note added: "VCCQ 1V8: 4u7 + 100n"
- note added: "VDDi: 2u2 (1-4.7 u)"
- note added: "e-MMC on SD0 (MIO40-45, bank 501, 1.8 V), 4-bit. Pull-ups to 1V8 (= VCCQ, the same supply as VCCO_MIO1, as the data sheet requires). RST_n pull-up = the MIO7 strap on sheet 6. R1001 (CLK, 0 R) sits at the MIO pin."

Commit message: LCSC numbers for every BOM part (tools/set_lcsc.py); FB1 as 0 R; U20 = XC7Z020-2CLG484I
tools/set_lcsc.py (run by build_schematic.sh) writes the LCSC field by BOM line: JLC basic parts where there is one,
juliancoy's Murata/Yageo passives bought as basic equivalents (REUSE_LOG E11). FB1, the E5 0 R jumper, gets
0603WAF0000T5E / C21189 (its MPN still named the bead). U20: -2 or -3 speed, any temperature grade (user):
XC7Z020-2CLG484I, C157624. Connectors J1/J2/J3/J5/J6/J9 hand-soldered (no LCSC, skipped in the JLC files).
ERC unchanged (4 intended pin_to_pin), block netlist 0 failures, board rebuilt: parity 0, block copper 0 failures.

Co-Authored-By: Claude Opus 5.5 <noreply@anthropic.com>
Parts:
- C1001, C1003: LCSC (none) -> C23733
- C1002: LCSC (none) -> C16772
- C1004: LCSC (none) -> C1525
- C1005: LCSC (none) -> C12530
- R1001: LCSC (none) -> C17168
- R1010, R1011, R1012, R1013, R1014, R1015, R1016, R1017, R1018, R1019: LCSC (none) -> C25792
Changed lines of the file:
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@@
+			)
+		)
+		(property "LCSC" "C17168"
+			(at 50.8 63.5 0)
+			(effects
+				(font
+					(size 1.27 1.27)
+				)
+				(hide yes)
 			)
 		)
@@
 			)
 		)
+		(property "LCSC" "C25792"
+			(at 38.1 154.94 0)
+			(effects
+				(font
+					(size 1.27 1.27)
+				)
+				(hide yes)
+			)
+		)
 		(property "Description" "Resistor"
 			(at 38.1 154.94 0)
@@
 			)
 		)
+		(property "LCSC" "C25792"
+			(at 48.26 154.94 0)
+			(effects
+				(font
+					(size 1.27 1.27)
+				)
+				(hide yes)
+			)
+		)
 		(property "Description" "Resistor"
 			(at 48.26 154.94 0)
@@
 			)
 		)
+		(property "LCSC" "C25792"
+			(at 58.42 154.94 0)
+			(effects
+				(font
+					(size 1.27 1.27)
+				)
+				(hide yes)
+			)
+		)
 		(property "Description" "Resistor"
 			(at 58.42 154.94 0)
@@
 			)
 		)
+		(property "LCSC" "C25792"
+			(at 68.58 154.94 0)
+			(effects
+				(font
+					(size 1.27 1.27)
+				)
+				(hide yes)
+			)
+		)
 		(property "Description" "Resistor"
 			(at 68.58 154.94 0)
@@
 			)
 		)
+		(property "LCSC" "C25792"
+			(at 78.74 154.94 0)
+			(effects
+				(font
+					(size 1.27 1.27)
+				)
+				(hide yes)
+			)
+		)
 		(property "Description" "Resistor"
 			(at 78.74 154.94 0)
@@
 			)
 		)
+		(property "LCSC" "C25792"
+			(at 88.9 154.94 0)
+			(effects
+				(font
+					(size 1.27 1.27)
+				)
+				(hide yes)
+			)
+		)
 		(property "Description" "Resistor"
 			(at 88.9 154.94 0)
@@
 			)
 		)
+		(property "LCSC" "C25792"
+			(at 99.06 154.94 0)
+			(effects
+				(font
+					(size 1.27 1.27)
+				)
+				(hide yes)
+			)
+		)
 		(property "Description" "Resistor"
 			(at 99.06 154.94 0)
@@
 			)
 		)
+		(property "LCSC" "C25792"
+			(at 109.22 154.94 0)
+			(effects
+				(font
+					(size 1.27 1.27)
+				)
+				(hide yes)
+			)
+		)
 		(property "Description" "Resistor"
 			(at 109.22 154.94 0)
@@
 			)
 		)
+		(property "LCSC" "C25792"
+			(at 119.38 154.94 0)
+			(effects
+				(font
+					(size 1.27 1.27)
+				)
+				(hide yes)
+			)
+		)
 		(property "Description" "Resistor"
 			(at 119.38 154.94 0)
@@
 			)
 		)
+		(property "LCSC" "C25792"
+			(at 129.54 154.94 0)
+			(effects
+				(font
+					(size 1.27 1.27)
+				)
+				(hide yes)
+			)
+		)
 		(property "Description" "Resistor"
 			(at 129.54 154.94 0)
@@
 		)
 		(property "Datasheet" ""
+			(at 38.1 203.2 0)
+			(effects
+				(font
+					(size 1.27 1.27)
+				)
+				(hide yes)
+			)
+		)
+		(property "LCSC" "C23733"
 			(at 38.1 203.2 0)
 			(effects
@@
 			)
 		)
+		(property "LCSC" "C16772"
+			(at 46.99 203.2 0)
+			(effects
+				(font
+					(size 1.27 1.27)
+				)
+				(hide yes)
+			)
+		)
 		(property "Description" "Unpolarized capacitor"
 			(at 46.99 203.2 0)
@@
 		)
 		(property "Datasheet" ""
+			(at 114.3 203.2 0)
+			(effects
+				(font
+					(size 1.27 1.27)
+				)
+				(hide yes)
+			)
+		)
+		(property "LCSC" "C23733"
 			(at 114.3 203.2 0)
 			(effects
@@
 			)
 		)
+		(property "LCSC" "C1525"
+			(at 123.19 203.2 0)
+			(effects
+				(font
+					(size 1.27 1.27)
+				)
+				(hide yes)
+			)
+		)
 		(property "Description" "Unpolarized capacitor"
 			(at 123.19 203.2 0)
@@
 			(at 190.5 203.2 0)
 			(effects
+				(font
+					(size 1.27 1.27)
+				)
+				(hide yes)
+			)
+		)
+		(property "LCSC" "C12530"
+			(at 190.5 203.2 0)
+			(effects
