File: kicad/11_soc_pl.kicad_sch (KiCad schematic)
At the start: 0 parts

Commit message: Phase 2: sheet 11 (PL banks 13/33/34/35, all VCCO on 3V3)
U20 units 2-5 with one hierarchical label per pin-plan signal (ball and
pin function asserted against the symbol); unused balls left open.
PUDC_B (K16) tied to VCCO_34; user LEDs D1101/D1102 on bank 33.
New block change E9: juliancoy grounds every I/O ball of banks 34/35;
here they carry our nets or stay open (copper planned). The block check
covers sheet 11, with E7/E9 balls generated from the symbol: 0 failures,
322 U20 balls. All 52 pin-plan signals verified on their balls.

Co-Authored-By: Claude Opus 5.5 <noreply@anthropic.com>
Parts:
- added D1101, D1102: red, LED_SMD:LED_0603_1608Metric, symbol zynq_card:LED
- added R1101, R1102: 1k, Resistor_SMD:R_0402_1005Metric, symbol zynq_card:R
- added U20: XC7Z020-1CLG484I, DFTcustom:BGA-484_19.0x19.0mm_Layout22x22_P0.80mm_dia0.40mm, symbol zynq_card:XC7Z020-CLG484
Connections:
- new net: D1101.2 (A), R1101.2
- new net: D1102.2 (A), R1102.2
- new net 3V3: R1101.1, R1102.1, U20.A20 (VCCO_35[7]), U20.AA10 (VCCO_13[7]), U20.AA20 (VCCO_33[6]), U20.AB13 (VCCO_33[6]), U20.AB3 (VCCO_13[7]), U20.C16 (VCCO_35[7]), U20.D19 (VCCO_35[7]), U20.E22 (VCCO_35[7]), U20.F15 (VCCO_35[7]), U20.G18 (VCCO_35[7]), U20.H21 (VCCO_35[7]), U20.K16 (IO_L3P_T0_DQS_PUDC_B_34), U20.K17 (VCCO_34[6]), U20.L20 (VCCO_34[6]), U20.N16 (VCCO_34[6]), U20.P19 (VCCO_34[6]), U20.R22 (VCCO_34[6]), U20.T15 (VCCO_34[6]), U20.T5 (VCCO_13[7]), U20.U18 (VCCO_33[6]), U20.U8 (VCCO_13[7]), U20.V11 (VCCO_13[7]), U20.V21 (VCCO_33[6]), U20.W14 (VCCO_33[6]), U20.W4 (VCCO_13[7]), U20.Y17 (VCCO_33[6]), U20.Y7 (VCCO_13[7])
- new net adasel0_iso: U20.J22 (IO_L8N_T1_34)
- new net adasel1_iso: U20.L22 (IO_L10N_T1_34)
- new net adasel2_iso: U20.M22 (IO_L15N_T2_DQS_34)
- new net adbsel0: U20.W22 (IO_L3N_T0_DQS_33)
- new net adbsel1: U20.AA22 (IO_L7P_T1_33)
- new net adbsel2: U20.AB22 (IO_L7N_T1_33)
- new net adc_cs_n: U20.T22 (IO_L2P_T0_33)
- new net adc_sclk: U20.U22 (IO_L2N_T0_33)
- new net adc_sdo: U20.V22 (IO_L3P_T0_DQS_33)
- new net adclk_dab: U20.P22 (IO_L16N_T2_34)
- new net adclk_iso: U20.N22 (IO_L16P_T2_34)
- new net clk1_iso: U20.K21 (IO_L9N_T1_DQS_34)
- new net cs1_iso: U20.L21 (IO_L10P_T1_34)
- new net dab_pwm_hi_sec: U20.J17 (IO_L2N_T0_34)
- new net dab_pwm_lo_sec: U20.L17 (IO_L4P_T0_34)
- new net dab_pwm_pri_hi_iso: U20.R18 (IO_L23P_T3_34)
- new net dab_pwm_pri_lo_iso: U20.T18 (IO_L23N_T3_34)
- new net gpio_bypass_rly_iso: U20.P21 (IO_L18N_T2_34)
- new net gpio_bypass_rly_isolated: U20.M21 (IO_L15P_T2_DQS_34)
- new net inu_adclk: U20.J21 (IO_L8P_T1_34)
- new net lcd_cs_n: U20.T21 (IO_L1P_T0_33)
- new net lcd_dc: U20.W21 (IO_L4N_T0_33)
- new net lcd_led: U20.AB21 (IO_L8N_T1_33)
- new net lcd_miso: U20.U20 (IO_L5P_T0_33)
- new net lcd_mosi: U20.AA21 (IO_L8P_T1_33)
- new net lcd_reset_n: U20.U21 (IO_L1N_T0_33)
- new net lcd_sck: U20.Y21 (IO_L9N_T1_DQS_33)
- new net led0_n: D1101.1 (K), U20.AB19 (IO_L10P_T1_33)
- new net led1_n: D1102.1 (K), U20.V18 (IO_L6P_T0_33)
- new net mdata_dab: U20.P16 (IO_L24P_T3_34)
- new net mdata_inu: U20.R16 (IO_L24N_T3_34)
- new net mdata_iso: U20.J16 (IO_L2P_T0_34)
- new net pwm_g1_iso: U20.J18 (IO_L7P_T1_34)
- new net pwm_g2_iso: U20.K18 (IO_L7N_T1_34)
- new net pwm_g3_iso: U20.N18 (IO_L5N_T0_34)
- new net pwm_g4_iso: U20.P18 (IO_L20N_T3_34)
- new net pwm_q5: U20.M17 (IO_L4N_T0_34)
- new net pwm_q6: U20.N17 (IO_L5P_T0_34)
- new net pwm_q7: U20.P17 (IO_L20P_T3_34)
- new net pwm_q8: U20.T17 (IO_L21N_T3_DQS_34)
- new net pwm_trans1_iso: U20.R21 (IO_L17N_T2_34)
- new net pwm_trans2_iso: U20.J20 (IO_L9P_T1_DQS_34)
- new net pwm_trans3_iso: U20.P20 (IO_L18P_T2_34)
- new net pwm_trans4: U20.R20 (IO_L17P_T2_34)
- new net pwm_trans5: U20.R19 (IO_L22P_T3_34)
- new net pwm_trans6: U20.T19 (IO_L22N_T3_34)
- new net sdata1_iso: U20.L16 (IO_L3N_T0_DQS_34)
- new net t_clk: U20.W20 (IO_L4P_T0_33)
- new net t_cs_n: U20.V20 (IO_L5N_T0_33)
- new net t_din: U20.Y20 (IO_L9P_T1_DQS_33)
- new net t_do: U20.AB20 (IO_L10N_T1_33)
- new net t_irq: U20.U19 (IO_0_33)
- no-connect marks 0 -> 147
Other:
- note added: "Bank 13: VCCO_13 = 3V3"
- note added: "Bank 33: VCCO_33 = 3V3"
- note added: "Bank 34: VCCO_34 = 3V3"
- note added: "Bank 35: VCCO_35 = 3V3"
- note added: "PUDC_B (K16) tied to VCCO_34 (UG865: directly or <= 1 k): no internal pull-ups during configuration; J3 pull-downs on sheet 13 hold the baseboard inputs low (J3 safe state)."
- note added: "U20 PL banks 13, 33, 34, 35: HR I/O, all at 3.3 V (LVCMOS33). Signal <-> ball from vivado/pinplan/pinplan.py (zynq_pinplan.csv, Vivado DRC 0). Change pins there, then re-run this script. Unused balls are left open. Bank 34 = J3 (pull-downs on sheet 13), bank 33 = ADC, LCD/touch, LEDs; banks 13 and 35 spare."
- note added: "User LEDs on bank 33 (active low)"

Commit message: LCSC numbers for every BOM part (tools/set_lcsc.py); FB1 as 0 R; U20 = XC7Z020-2CLG484I
tools/set_lcsc.py (run by build_schematic.sh) writes the LCSC field by BOM line: JLC basic parts where there is one,
juliancoy's Murata/Yageo passives bought as basic equivalents (REUSE_LOG E11). FB1, the E5 0 R jumper, gets
0603WAF0000T5E / C21189 (its MPN still named the bead). U20: -2 or -3 speed, any temperature grade (user):
XC7Z020-2CLG484I, C157624. Connectors J1/J2/J3/J5/J6/J9 hand-soldered (no LCSC, skipped in the JLC files).
ERC unchanged (4 intended pin_to_pin), block netlist 0 failures, board rebuilt: parity 0, block copper 0 failures.

Co-Authored-By: Claude Opus 5.5 <noreply@anthropic.com>
Parts:
- D1101, D1102: LCSC (none) -> C2286; MPN (none) -> KT-0603R
- R1101, R1102: LCSC (none) -> C11702
- U20: value XC7Z020-1CLG484I -> XC7Z020-2CLG484I; LCSC (none) -> C157624; MPN (none) -> XC7Z020-2CLG484I
Changed lines of the file:
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@@
 			)
 		)
-		(property "Value" "XC7Z020-1CLG484I"
+		(property "Value" "XC7Z020-2CLG484I"
 			(at 58.42 46.99 0)
 			(effects
@@
 		)
 		(property "Datasheet" ""
+			(at 58.42 50.8 0)
+			(effects
+				(font
+					(size 1.27 1.27)
+				)
+				(hide yes)
+			)
+		)
+		(property "LCSC" "C157624"
+			(at 58.42 50.8 0)
+			(effects
+				(font
+					(size 1.27 1.27)
+				)
+				(hide yes)
+			)
+		)
+		(property "MPN" "XC7Z020-2CLG484I"
 			(at 58.42 50.8 0)
 			(effects
@@
 			)
 		)
-		(property "Value" "XC7Z020-1CLG484I"
+		(property "Value" "XC7Z020-2CLG484I"
 			(at 157.48 46.99 0)
 			(effects
@@
 		)
 		(property "Datasheet" ""
+			(at 157.48 50.8 0)
+			(effects
+				(font
+					(size 1.27 1.27)
+				)
+				(hide yes)
+			)
+		)
+		(property "LCSC" "C157624"
+			(at 157.48 50.8 0)
+			(effects
+				(font
+					(size 1.27 1.27)
+				)
+				(hide yes)
+			)
+		)
+		(property "MPN" "XC7Z020-2CLG484I"
 			(at 157.48 50.8 0)
 			(effects
@@
 			)
 		)
-		(property "Value" "XC7Z020-1CLG484I"
+		(property "Value" "XC7Z020-2CLG484I"
 			(at 256.54 46.99 0)
 			(effects
@@
 		)
 		(property "Datasheet" ""
+			(at 256.54 50.8 0)
+			(effects
+				(font
+					(size 1.27 1.27)
+				)
+				(hide yes)
+			)
+		)
+		(property "LCSC" "C157624"
+			(at 256.54 50.8 0)
+			(effects
+				(font
+					(size 1.27 1.27)
+				)
+				(hide yes)
+			)
+		)
+		(property "MPN" "XC7Z020-2CLG484I"
 			(at 256.54 50.8 0)
 			(effects
@@
 			)
 		)
-		(property "Value" "XC7Z020-1CLG484I"
+		(property "Value" "XC7Z020-2CLG484I"
 			(at 355.6 46.99 0)
 			(effects
@@
 		)
 		(property "Datasheet" ""
+			(at 355.6 50.8 0)
+			(effects
+				(font
+					(size 1.27 1.27)
+				)
+				(hide yes)
+			)
+		)
+		(property "LCSC" "C157624"
+			(at 355.6 50.8 0)
+			(effects
+				(font
+					(size 1.27 1.27)
+				)
+				(hide yes)
+			)
+		)
+		(property "MPN" "XC7Z020-2CLG484I"
 			(at 355.6 50.8 0)
 			(effects
@@
 			)
 		)
+		(property "LCSC" "C11702"
+			(at 177.8 243.84 0)
+			(effects
+				(font
+					(size 1.27 1.27)
+				)
+				(hide yes)
+			)
+		)
 		(property "Description" "Resistor"
 			(at 177.8 243.84 0)
@@
 			)
 		)
+		(property "MPN" "KT-0603R"
+			(at 177.8 254 0)
+			(effects
+				(font
+					(size 1.27 1.27)
+				)
+				(hide yes)
+			)
+		)
+		(property "LCSC" "C2286"
+			(at 177.8 254 0)
+			(effects
+				(font
+					(size 1.27 1.27)
+				)
+				(hide yes)
+			)
+		)
 		(property "Description" "Light emitting diode"
 			(at 177.8 254 0)
@@
 			)
 		)
+		(property "LCSC" "C11702"
+			(at 195.58 243.84 0)
+			(effects
+				(font
+					(size 1.27 1.27)
+				)
+				(hide yes)
+			)
+		)
 		(property "Description" "Resistor"
 			(at 195.58 243.84 0)
@@
 			(at 195.58 254 0)
 			(effects
+				(font
+					(size 1.27 1.27)
+				)
+				(hide yes)
+			)
+		)
+		(property "MPN" "KT-0603R"
+			(at 195.58 254 0)
+			(effects
+				(font
+					(size 1.27 1.27)
+				)
+				(hide yes)
+			)
+		)
+		(property "LCSC" "C2286"
+			(at 195.58 254 0)
+			(effects
