File: kicad/12_adc.kicad_sch (KiCad schematic)
At the start: 0 parts

Commit message: Phase 2: sheets 12-13 (ADC, connectors) + pin-plan netlist check
- Sheet 12: Ti135 ADC chain (SN74LV4051A checked against SCLS428K, OPA365,
  ADS7056 with AVDD on 3V3_analog and DVDD on 3V3), selects/SPI straight to bank 33.
- Sheet 13: J3 (baseboard J11 numbering, pin-plan notes asserted) with 32 x 10 k
  pull-downs, J5 LCD/touch, J2 console via SN74AVC4T774 (per-bit direction),
  I2C0 4.7 k pull-ups to 1V8 (no EEPROM for now).
- tools/check_pinplan_netlist.py: every PL and MIO signal on its ball: 0 failures.
- ERC: 4 expected pin_to_pin ties; block check 0 failures.

Co-Authored-By: Claude Opus 5.5 <noreply@anthropic.com>
Parts:
- added C1201, C1206: 1u, Capacitor_SMD:C_0402_1005Metric, symbol zynq_card:C
- added C1202: 680p C0G, Capacitor_SMD:C_0402_1005Metric, symbol zynq_card:C
- added C1203, C1205: 100n, Capacitor_SMD:C_0402_1005Metric, symbol zynq_card:C
- added C1204: 4u7, Capacitor_SMD:C_0603_1608Metric, symbol zynq_card:C
- added R1201: 100R, Resistor_SMD:R_0402_1005Metric, symbol zynq_card:R
- added R1202, R1203, R1204, R1205: 1k, Resistor_SMD:R_0402_1005Metric, symbol zynq_card:R
- added R1206, R1210, R1211, R1212: 33R, Resistor_SMD:R_0402_1005Metric, symbol zynq_card:R
- added U1201: SN74LV4051APWR, Package_SO:TSSOP-16_4.4x5mm_P0.65mm, symbol zynq_card:CD4051B
- added U1202: OPA365AIDBVR, Package_TO_SOT_SMD:SOT-23-5, symbol zynq_card:OPA365xxDBV
- added U1203: ADS7056IRUGR, zynq_card:ads7056, symbol zynq_card:ADS7056
Connections:
- new net: R1206.1, U1202.1, U1202.4 (-)
- new net 1V0: R1201.1
- new net 1V35: R1204.1
- new net 1V8: R1202.1
- new net 3V3: C1206.1, R1203.1, U1203.4 (DVDD)
- new net 3V3_analog: C1201.1, C1203.1, C1204.1, C1205.1, U1201.16 (VDD), U1202.5 (V+), U1203.6 (AVDD)
- new net GND: C1201.2, C1202.2, C1203.2, C1204.2, C1205.2, C1206.2, R1205.2, U1201.13 (X0), U1201.6 (INH), U1201.7 (VEE), U1201.8 (VSS), U1202.2 (V-), U1203.5 (GND), U1203.8 (AINM)
- new net adbsel0: U1201.11 (A)
- new net adbsel1: U1201.10 (B)
- new net adbsel2: U1201.9 (C)
- new net adc_ainp: C1202.1, R1206.2, U1203.7 (AINP)
- new net adc_cs_n: R1210.1
- new net adc_cs_n_r: R1210.2, U1203.1 (~{CS})
- new net adc_mux_out: U1201.3 (X), U1202.3 (+)
- new net adc_sclk: R1211.1
- new net adc_sclk_r: R1211.2, U1203.3 (SCLK)
- new net adc_sdo: R1212.1
- new net adc_sdo_r: R1212.2, U1203.2 (SDO)
- new net isoada1: U1201.4 (X7)
- new net isoada2: U1201.1 (X4)
- new net isoada3: U1201.2 (X6)
- new net mon_1v0: R1201.2, U1201.14 (X1)
- new net mon_1v35: R1204.2, U1201.5 (X5)
- new net mon_1v8: R1202.2, U1201.15 (X2)
- new net mon_3v3: R1203.2, R1205.1, U1201.12 (X3)
Other:
- note added: "3V3 via 1k/1k divider"
- note added: "ADC chain: mux U1201 -> buffer U1202 -> ADS7056 U1203 (Ti135 sheet 13; front end as on the Agilex 3 card, 2.5 MSPS). Mux: X0 GND (zero ref), X1 1V0, X2 1V8, X3 3V3/2, X4 isoada2, X5 1V35, X6 isoada3, X7 isoada1. Full scale 0..3.3 V (AVDD = reference, 3V3_analog). DVDD on 3V3: SPI and selects straight to bank 33."
- note added: "AVDD = reference: 4u7 0603 + 100n at the pin"
- note added: "DVDD 3V3"
- note added: "Rail monitors"
- note added: "SN74LV4051A (SCLS428K): pins 7/8 GND; VIH 2.31 V at 3.3 V"
- note added: "SPI series 33 R (60 MHz SCLK); DVDD 3V3 = bank 33"
- note added: "U1201 VCC"
- note added: "U1202 V+"

Commit message: LCSC numbers for every BOM part (tools/set_lcsc.py); FB1 as 0 R; U20 = XC7Z020-2CLG484I
tools/set_lcsc.py (run by build_schematic.sh) writes the LCSC field by BOM line: JLC basic parts where there is one,
juliancoy's Murata/Yageo passives bought as basic equivalents (REUSE_LOG E11). FB1, the E5 0 R jumper, gets
0603WAF0000T5E / C21189 (its MPN still named the bead). U20: -2 or -3 speed, any temperature grade (user):
XC7Z020-2CLG484I, C157624. Connectors J1/J2/J3/J5/J6/J9 hand-soldered (no LCSC, skipped in the JLC files).
ERC unchanged (4 intended pin_to_pin), block netlist 0 failures, board rebuilt: parity 0, block copper 0 failures.

Co-Authored-By: Claude Opus 5.5 <noreply@anthropic.com>
Parts:
- C1201, C1206: LCSC (none) -> C52923
- C1202: LCSC (none) -> C113781
- C1203, C1205: LCSC (none) -> C1525
- C1204: LCSC (none) -> C19666
- R1201: LCSC (none) -> C25076
- R1202, R1203, R1204, R1205: LCSC (none) -> C11702
- R1206, R1210, R1211, R1212: LCSC (none) -> C25105
Changed lines of the file:
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@@
 			)
 		)
+		(property "LCSC" "C52923"
+			(at 76.2 152.4 0)
+			(effects
+				(font
+					(size 1.27 1.27)
+				)
+				(hide yes)
+			)
+		)
 		(property "Description" "Unpolarized capacitor"
 			(at 76.2 152.4 0)
@@
 			)
 		)
+		(property "LCSC" "C25076"
+			(at 22.86 193.04 0)
+			(effects
+				(font
+					(size 1.27 1.27)
+				)
+				(hide yes)
+			)
+		)
 		(property "Description" "Resistor"
 			(at 22.86 193.04 0)
@@
 			)
 		)
+		(property "LCSC" "C11702"
+			(at 33.02 193.04 0)
+			(effects
+				(font
+					(size 1.27 1.27)
+				)
+				(hide yes)
+			)
+		)
 		(property "Description" "Resistor"
 			(at 33.02 193.04 0)
@@
 			)
 		)
+		(property "LCSC" "C11702"
+			(at 43.18 193.04 0)
+			(effects
+				(font
+					(size 1.27 1.27)
+				)
+				(hide yes)
+			)
+		)
 		(property "Description" "Resistor"
 			(at 43.18 193.04 0)
@@
 			)
 		)
+		(property "LCSC" "C11702"
+			(at 53.34 193.04 0)
+			(effects
+				(font
+					(size 1.27 1.27)
+				)
+				(hide yes)
+			)
+		)
 		(property "Description" "Resistor"
 			(at 53.34 193.04 0)
@@
 			)
 		)
+		(property "LCSC" "C11702"
+			(at 63.5 193.04 0)
+			(effects
+				(font
+					(size 1.27 1.27)
+				)
+				(hide yes)
+			)
+		)
 		(property "Description" "Resistor"
 			(at 63.5 193.04 0)
@@
 			)
 		)
+		(property "LCSC" "C25105"
+			(at 223.52 101.6 0)
+			(effects
+				(font
+					(size 1.27 1.27)
+				)
+				(hide yes)
+			)
+		)
 		(property "Description" "Resistor"
 			(at 223.52 101.6 0)
@@
 			)
 		)
+		(property "LCSC" "C113781"
+			(at 232.41 107.95 0)
+			(effects
+				(font
+					(size 1.27 1.27)
+				)
+				(hide yes)
+			)
+		)
 		(property "Description" "Unpolarized capacitor"
 			(at 232.41 107.95 0)
@@
 			)
 		)
+		(property "LCSC" "C1525"
+			(at 190.5 152.4 0)
+			(effects
+				(font
+					(size 1.27 1.27)
+				)
+				(hide yes)
+			)
+		)
 		(property "Description" "Unpolarized capacitor"
 			(at 190.5 152.4 0)
@@
 			)
 		)
+		(property "LCSC" "C19666"
+			(at 292.1 152.4 0)
+			(effects
+				(font
+					(size 1.27 1.27)
+				)
+				(hide yes)
+			)
+		)
 		(property "Description" "Unpolarized capacitor"
 			(at 292.1 152.4 0)
@@
 			)
 		)
+		(property "LCSC" "C1525"
+			(at 300.99 152.4 0)
+			(effects
+				(font
+					(size 1.27 1.27)
+				)
+				(hide yes)
+			)
+		)
 		(property "Description" "Unpolarized capacitor"
 			(at 300.99 152.4 0)
@@
 			)
 		)
+		(property "LCSC" "C52923"
+			(at 368.3 152.4 0)
+			(effects
+				(font
+					(size 1.27 1.27)
+				)
+				(hide yes)
+			)
+		)
 		(property "Description" "Unpolarized capacitor"
 			(at 368.3 152.4 0)
@@
 			)
 		)
+		(property "LCSC" "C25105"
+			(at 304.8 187.96 0)
+			(effects
+				(font
+					(size 1.27 1.27)
+				)
+				(hide yes)
+			)
+		)
 		(property "Description" "Resistor"
 			(at 304.8 187.96 0)
@@
 			)
 		)
+		(property "LCSC" "C25105"
+			(at 304.8 194.31 0)
+			(effects
+				(font
+					(size 1.27 1.27)
+				)
+				(hide yes)
+			)
+		)
 		(property "Description" "Resistor"
 			(at 304.8 194.31 0)
@@
 			(at 304.8 200.66 0)
 			(effects
+				(font
+					(size 1.27 1.27)
+				)
+				(hide yes)
+			)
+		)
+		(property "LCSC" "C25105"
+			(at 304.8 200.66 0)
+			(effects
