File: kicad/13_connectors.kicad_sch (KiCad schematic)
At the start: 0 parts

Commit message: Phase 2: sheets 12-13 (ADC, connectors) + pin-plan netlist check
- Sheet 12: Ti135 ADC chain (SN74LV4051A checked against SCLS428K, OPA365,
  ADS7056 with AVDD on 3V3_analog and DVDD on 3V3), selects/SPI straight to bank 33.
- Sheet 13: J3 (baseboard J11 numbering, pin-plan notes asserted) with 32 x 10 k
  pull-downs, J5 LCD/touch, J2 console via SN74AVC4T774 (per-bit direction),
  I2C0 4.7 k pull-ups to 1V8 (no EEPROM for now).
- tools/check_pinplan_netlist.py: every PL and MIO signal on its ball: 0 failures.
- ERC: 4 expected pin_to_pin ties; block check 0 failures.

Co-Authored-By: Claude Opus 5.5 <noreply@anthropic.com>
Parts:
- added C1301, C1302: 100n, Capacitor_SMD:C_0402_1005Metric, symbol zynq_card:C
- added J2: UART 3V3, Connector_PinHeader_2.54mm:PinHeader_1x03_P2.54mm_Vertical, symbol zynq_card:Conn_01x03
- added J3: 2x19 1.27mm socket (bottom), Connector_PinSocket_1.27mm:PinSocket_2x19_P1.27mm_Vertical, symbol zynq_card:Conn_02x19_Odd_Even
- added J5: LCD 1x14 2.54mm, Connector_PinHeader_2.54mm:PinHeader_1x14_P2.54mm_Vertical, symbol zynq_card:Conn_01x14
- added R1301, R1302: 1k, Resistor_SMD:R_0402_1005Metric, symbol zynq_card:R
- added R1303, R1304: 10k, Resistor_SMD:R_0402_1005Metric, symbol zynq_card:R
- added R1305, R1306: 4.7k, Resistor_SMD:R_0402_1005Metric, symbol zynq_card:R
- added RN1301, RN1302, RN1303, RN1304, RN1305, RN1306, RN1307, RN1308: 4x10k, Resistor_SMD:R_Array_Convex_4x0402, symbol zynq_card:R_Pack04
- added U1301: SN74AVC4T774RSVR, Package_DFN_QFN:UQFN-16_1.8x2.6mm_P0.4mm, symbol zynq_card:SN74AVC4T774
Connections:
- new net: J2.1 (Pin_1), R1301.2
- new net: J2.2 (Pin_2), R1302.2
- new net 1V8: C1302.1, R1304.1, R1305.1, R1306.1, U1301.13 (VCCB)
- new net 3V3: C1301.1, J5.14 (Pin_14), R1303.1, U1301.14 (VCCA), U1301.15 (DIR1), U1301.5 (DIR3), U1301.6 (DIR4)
- new net GND: C1301.2, C1302.2, J2.3 (Pin_3), J3.2 (Pin_2), J3.5 (Pin_5), J5.13 (Pin_13), RN1301.5 (R4.2), RN1301.6 (R3.2), RN1301.7 (R2.2), RN1301.8 (R1.2), RN1302.5 (R4.2), RN1302.6 (R3.2), RN1302.7 (R2.2), RN1302.8 (R1.2), RN1303.5 (R4.2), RN1303.6 (R3.2), RN1303.7 (R2.2), RN1303.8 (R1.2), RN1304.5 (R4.2), RN1304.6 (R3.2), RN1304.7 (R2.2), RN1304.8 (R1.2), RN1305.5 (R4.2), RN1305.6 (R3.2), RN1305.7 (R2.2), RN1305.8 (R1.2), RN1306.5 (R4.2), RN1306.6 (R3.2), RN1306.7 (R2.2), RN1306.8 (R1.2), RN1307.5 (R4.2), RN1307.6 (R3.2), RN1307.7 (R2.2), RN1307.8 (R1.2), RN1308.5 (R4.2), RN1308.6 (R3.2), RN1308.7 (R2.2), RN1308.8 (R1.2), U1301.16 (DIR2), U1301.3 (A3), U1301.4 (A4), U1301.7 (~{OE}), U1301.8 (GND)
- new net adasel0_iso: J3.11 (Pin_11), RN1302.2 (R2.1)
- new net adasel1_iso: J3.10 (Pin_10), RN1302.1 (R1.1)
- new net adasel2_iso: J3.9 (Pin_9), RN1301.4 (R4.1)
- new net adclk_dab: J3.24 (Pin_24), RN1305.3 (R3.1)
- new net adclk_iso: J3.7 (Pin_7), RN1301.2 (R2.1)
- new net clk1_iso: J3.14 (Pin_14), RN1303.1 (R1.1)
- new net cs1_iso: J3.13 (Pin_13), RN1302.4 (R4.1)
- new net dab_pwm_hi_sec: J3.27 (Pin_27), RN1306.2 (R2.1)
- new net dab_pwm_lo_sec: J3.29 (Pin_29), RN1306.4 (R4.1)
- new net dab_pwm_pri_hi_iso: J3.22 (Pin_22), RN1305.1 (R1.1)
- new net dab_pwm_pri_lo_iso: J3.23 (Pin_23), RN1305.2 (R2.1)
- new net gpio_bypass_rly_iso: J3.36 (Pin_36), RN1308.3 (R3.1)
- new net gpio_bypass_rly_isolated: J3.8 (Pin_8), RN1301.3 (R3.1)
- new net i2c_scl: R1305.2
- new net i2c_sda: R1306.2
- new net inu_adclk: J3.32 (Pin_32), RN1307.3 (R3.1)
- new net isoada1: J3.4 (Pin_4)
- new net isoada2: J3.3 (Pin_3)
- new net isoada3: J3.1 (Pin_1)
- new net lcd_cs_n: J5.12 (Pin_12)
- new net lcd_dc: J5.10 (Pin_10)
- new net lcd_led: J5.7 (Pin_7)
- new net lcd_miso: J5.9 (Pin_9)
- new net lcd_mosi: J5.6 (Pin_6)
- new net lcd_reset_n: J5.11 (Pin_11)
- new net lcd_sck: J5.8 (Pin_8)
- new net mdata_dab: J3.26 (Pin_26), RN1306.1 (R1.1)
- new net mdata_inu: J3.34 (Pin_34), RN1308.1 (R1.1)
- new net mdata_iso: J3.6 (Pin_6), RN1301.1 (R1.1)
- new net pwm_g1_iso: J3.20 (Pin_20), RN1304.3 (R3.1)
- new net pwm_g2_iso: J3.19 (Pin_19), RN1304.2 (R2.1)
- new net pwm_g3_iso: J3.21 (Pin_21), RN1304.4 (R4.1)
- new net pwm_g4_iso: J3.18 (Pin_18), RN1304.1 (R1.1)
- new net pwm_q5: J3.30 (Pin_30), RN1307.1 (R1.1)
- new net pwm_q6: J3.31 (Pin_31), RN1307.2 (R2.1)
- new net pwm_q7: J3.37 (Pin_37), RN1308.4 (R4.1)
- new net pwm_q8: J3.33 (Pin_33), RN1307.4 (R4.1)
- new net pwm_trans1_iso: J3.15 (Pin_15), RN1303.2 (R2.1)
- new net pwm_trans2_iso: J3.16 (Pin_16), RN1303.3 (R3.1)
- new net pwm_trans3_iso: J3.17 (Pin_17), RN1303.4 (R4.1)
- new net pwm_trans4: J3.25 (Pin_25), RN1305.4 (R4.1)
- new net pwm_trans5: J3.35 (Pin_35), RN1308.2 (R2.1)
- new net pwm_trans6: J3.28 (Pin_28), RN1306.3 (R3.1)
- new net sdata1_iso: J3.12 (Pin_12), RN1302.3 (R3.1)
- new net t_clk: J5.5 (Pin_5)
- new net t_cs_n: J5.4 (Pin_4)
- new net t_din: J5.3 (Pin_3)
- new net t_do: J5.2 (Pin_2)
- new net t_irq: J5.1 (Pin_1)
- new net uart_rx: U1301.12 (B1)
- new net uart_rx_3v3: R1301.1, R1303.2, U1301.1 (A1)
- new net uart_tx: R1304.2, U1301.11 (B2)
- new net uart_tx_3v3: R1302.1, U1301.2 (A2)
- no-connect marks 0 -> 3
Other:
- note added: "I2C0 (MIO50 SCL, MIO51 SDA, 1.8 V): 4.7 k pull-ups to 1V8 (ZYNQ_PCB_NOTES.md §4.3). No device fitted yet."
- note added: "J2: 1 RX (into the SoC), 2 TX, 3 GND"
- note added: "J2: UART console (PS UART1, MIO48 TX / MIO49 RX, 1.8 V), family pinout 1 RX, 2 TX, 3 GND at 3.3 V. U1301 SN74AVC4T774RSVR (C779392), per-bit direction: A = J2 side (3V3), B = MIO side (1V8). DIR1 = H: J2 RX A1 -> B1; DIR2 = L: TX B2 -> A2; bits 3/4 unused (DIR H, A3/A4 to GND). OE low."
- note added: "J3 = baseboard J11 (2x19 1.27 mm socket on B.Cu, pin n = baseboard pin n, see MECHANICAL.md). Nets = sheet-11 names (bank 34, 3.3 V, no translators). Every digital pin has a 10 k pull-down: with PUDC_B high the PL has no pull-ups while unconfigured, so the baseboard sees low (J3 safe state). isoada1-3: analog, to the mux."
- note added: "J3 pull-downs: 8 x 4D02WGJ0103TCE (4 x 10 k, C25725)"
- note added: "J5: LCD/touch header, Ti135 J5 (Ti60 J4) pinout (wired to the LCD with jumper wires)."
- note added: "R1303: RX idle high with J2 open; R1304: B2 defined while MIO48 is off"
- note added: "VCCA"
- note added: "VCCB"

Commit message: LCSC numbers for every BOM part (tools/set_lcsc.py); FB1 as 0 R; U20 = XC7Z020-2CLG484I
tools/set_lcsc.py (run by build_schematic.sh) writes the LCSC field by BOM line: JLC basic parts where there is one,
juliancoy's Murata/Yageo passives bought as basic equivalents (REUSE_LOG E11). FB1, the E5 0 R jumper, gets
0603WAF0000T5E / C21189 (its MPN still named the bead). U20: -2 or -3 speed, any temperature grade (user):
XC7Z020-2CLG484I, C157624. Connectors J1/J2/J3/J5/J6/J9 hand-soldered (no LCSC, skipped in the JLC files).
ERC unchanged (4 intended pin_to_pin), block netlist 0 failures, board rebuilt: parity 0, block copper 0 failures.

Co-Authored-By: Claude Opus 5.5 <noreply@anthropic.com>
Parts:
- C1301, C1302: LCSC (none) -> C1525
- R1301, R1302: LCSC (none) -> C11702
- R1303, R1304: LCSC (none) -> C25744
- R1305, R1306: LCSC (none) -> C25900
Changed lines of the file:
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@@
+			)
+		)
+		(property "LCSC" "C1525"
+			(at 198.12 236.22 0)
+			(effects
+				(font
+					(size 1.27 1.27)
+				)
+				(hide yes)
 			)
 		)
@@
 			)
 		)
+		(property "LCSC" "C1525"
+			(at 241.3 236.22 0)
+			(effects
+				(font
+					(size 1.27 1.27)
+				)
+				(hide yes)
+			)
+		)
 		(property "Description" "Unpolarized capacitor"
 			(at 241.3 236.22 0)
@@
 		)
 		(property "Datasheet" ""
+			(at 147.32 200.66 0)
+			(effects
+				(font
+					(size 1.27 1.27)
+				)
+				(hide yes)
+			)
+		)
+		(property "LCSC" "C11702"
 			(at 147.32 200.66 0)
 			(effects
@@
 			)
 		)
+		(property "LCSC" "C11702"
+			(at 147.32 203.2 0)
+			(effects
+				(font
+					(size 1.27 1.27)
+				)
+				(hide yes)
+			)
+		)
 		(property "Description" "Resistor"
 			(at 147.32 203.2 0)
@@
 			)
 		)
+		(property "LCSC" "C25744"
+			(at 165.1 236.22 0)
+			(effects
+				(font
+					(size 1.27 1.27)
+				)
+				(hide yes)
+			)
+		)
 		(property "Description" "Resistor"
 			(at 165.1 236.22 0)
@@
 		)
 		(property "Datasheet" ""
+			(at 269.24 236.22 0)
+			(effects
+				(font
+					(size 1.27 1.27)
+				)
+				(hide yes)
+			)
+		)
+		(property "LCSC" "C25744"
 			(at 269.24 236.22 0)
 			(effects
@@
 			)
 		)
+		(property "LCSC" "C25900"
+			(at 342.9 203.2 0)
+			(effects
+				(font
+					(size 1.27 1.27)
+				)
+				(hide yes)
+			)
+		)
 		(property "Description" "Resistor"
 			(at 342.9 203.2 0)
@@
 			(at 358.14 203.2 0)
 			(effects
+				(font
+					(size 1.27 1.27)
+				)
+				(hide yes)
+			)
+		)
+		(property "LCSC" "C25900"
+			(at 358.14 203.2 0)
+			(effects
